File: vcu/drs-driver.kicad_sch (KiCad schematic)
At the start: 8 parts, among them U8 LTC6992-2

Commit message: feat(vcu): add test points to I2C bus
Parts:
- renumbered C14 to C7, R15 to R10, R16 to R11, R17 to R12, R13 to R8, R14 to R9, TP2 to TP15, U8 to U6
Changed lines of the file:
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@@
   (symbol (lib_id "power:GND") (at 132.08 108.585 0) (unit 1)
     (in_bom yes) (on_board yes)
-    (property "Reference" "#PWR056" (id 0) (at 132.08 114.935 0)
+    (property "Reference" "#PWR048" (id 0) (at 132.08 114.935 0)
       (effects (font (size 1.27 1.27)) hide)
     )
@@
   (symbol (lib_id "power:+5V") (at 173.99 93.345 0) (unit 1)
     (in_bom yes) (on_board yes)
-    (property "Reference" "#PWR0103" (id 0) (at 173.99 97.155 0)
+    (property "Reference" "#PWR050" (id 0) (at 173.99 97.155 0)
       (effects (font (size 1.27 1.27)) hide)
     )
@@
   (symbol (lib_id "Device:R_Small") (at 115.57 94.615 0) (unit 1)
     (in_bom yes) (on_board yes)
-    (property "Reference" "R14" (id 0) (at 116.84 93.345 0)
+    (property "Reference" "R9" (id 0) (at 116.84 93.345 0)
       (effects (font (size 1.27 1.27)) (justify left))
     )
@@
   (symbol (lib_id "Device:R_Small") (at 115.57 84.455 0) (unit 1)
     (in_bom yes) (on_board yes)
-    (property "Reference" "R13" (id 0) (at 116.84 83.185 0)
+    (property "Reference" "R8" (id 0) (at 116.84 83.185 0)
       (effects (font (size 1.27 1.27)) (justify left))
     )
@@
   (symbol (lib_id "power:GND") (at 162.56 102.235 0) (unit 1)
     (in_bom yes) (on_board yes)
-    (property "Reference" "#PWR057" (id 0) (at 162.56 108.585 0)
+    (property "Reference" "#PWR049" (id 0) (at 162.56 108.585 0)
       (effects (font (size 1.27 1.27)) hide)
     )
@@
   (symbol (lib_id "Device:R_Small") (at 132.08 104.14 0) (unit 1)
     (in_bom yes) (on_board yes)
-    (property "Reference" "R15" (id 0) (at 133.35 102.87 0)
+    (property "Reference" "R10" (id 0) (at 133.35 102.87 0)
       (effects (font (size 1.27 1.27)) (justify left))
     )
@@
   (symbol (lib_id "Device:R_Small") (at 173.99 100.965 0) (unit 1)
     (in_bom yes) (on_board yes)
-    (property "Reference" "R16" (id 0) (at 175.26 99.695 0)
+    (property "Reference" "R11" (id 0) (at 175.26 99.695 0)
       (effects (font (size 1.27 1.27)) (justify left))
     )
@@
   (symbol (lib_id "Device:C_Small") (at 162.56 98.425 0) (mirror y) (unit 1)
     (in_bom yes) (on_board yes)
-    (property "Reference" "C14" (id 0) (at 164.465 97.155 0)
+    (property "Reference" "C7" (id 0) (at 164.465 97.155 0)
       (effects (font (size 1.27 1.27)) (justify right))
     )
@@
   (symbol (lib_id "Connector:TestPoint_Small") (at 187.96 84.455 0) (unit 1)
     (in_bom yes) (on_board yes)
-    (property "Reference" "TP2" (id 0) (at 189.23 83.1849 0)
+    (property "Reference" "TP15" (id 0) (at 189.23 83.1849 0)
       (effects (font (size 1.27 1.27)) (justify left))
     )
@@
   (symbol (lib_id "power:GND") (at 115.57 98.425 0) (unit 1)
     (in_bom yes) (on_board yes)
-    (property "Reference" "#PWR054" (id 0) (at 115.57 104.775 0)
+    (property "Reference" "#PWR046" (id 0) (at 115.57 104.775 0)
       (effects (font (size 1.27 1.27)) hide)
     )
@@
   (symbol (lib_id "power:GND") (at 125.095 108.585 0) (unit 1)
     (in_bom yes) (on_board yes)
-    (property "Reference" "#PWR055" (id 0) (at 125.095 114.935 0)
+    (property "Reference" "#PWR047" (id 0) (at 125.095 114.935 0)
       (effects (font (size 1.27 1.27)) hide)
     )
@@
   (symbol (lib_id "symbols:LTC6992") (at 145.415 94.615 0) (unit 1)
     (in_bom yes) (on_board yes)
-    (property "Reference" "U8" (id 0) (at 145.415 85.725 0))
+    (property "Reference" "U6" (id 0) (at 145.415 85.725 0))
     (property "Value" "LTC6992-2" (id 1) (at 145.415 103.505 0))
     (property "Footprint" "Package_TO_SOT_SMD:SOT-23-6" (id 2) (at 145.415 94.615 0)
@@
   (symbol (lib_id "power:GND") (at 173.99 116.84 0) (unit 1)
     (in_bom yes) (on_board yes)
-    (property "Reference" "#PWR059" (id 0) (at 173.99 123.19 0)
+    (property "Reference" "#PWR051" (id 0) (at 173.99 123.19 0)
       (effects (font (size 1.27 1.27)) hide)
     )
@@
   (symbol (lib_id "Device:R_Small") (at 173.99 112.395 0) (unit 1)
     (in_bom yes) (on_board yes)
-    (property "Reference" "R17" (id 0) (at 175.26 111.125 0)
-      (effects (font (size 1.27 1.27)) (justify left))
-    )
+    (property "Reference" "R12" (id 0) (at 175.26 111.125 0)
+      (effects (font (size 1.27 1.27)) (justify left))
+    )
