File: vcu/input-shift.kicad_sch (KiCad schematic)
At the start: 26 parts, among them U4 ILQ615-4X009T

Commit message: chore(vcu): reset footprints
Parts:
- D2, D3, D4: footprint Package_TO_SOT_SMD:SOT-23 -> (none)
- R14, R15, R16, R17, R18, R19, R2, R3, R6, R7, R8, R9: footprint Resistor_SMD:R_0603_1608Metric_Pad0.98x0.95mm_HandSolder -> (none)
- RV2, RV3, RV4: footprint Potentiometer_THT:Potentiometer_Vishay_T73XW_Horizontal -> (none)
- TP10, TP11, TP9: footprint TestPoint:TestPoint_Pad_D1.5mm -> (none)
Changed lines of the file:
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@@
       (effects (font (size 1.27 1.27)) (justify right))
     )
-    (property "Footprint" "Resistor_SMD:R_0603_1608Metric_Pad0.98x0.95mm_HandSolder" (id 2) (at 40.005 119.38 0)
+    (property "Footprint" "" (id 2) (at 40.005 119.38 0)
       (effects (font (size 1.27 1.27)) hide)
     )
@@
       (effects (font (size 1.27 1.27)) (justify right))
     )
-    (property "Footprint" "Potentiometer_THT:Potentiometer_Vishay_T73XW_Horizontal" (id 2) (at 40.005 158.75 0)
+    (property "Footprint" "" (id 2) (at 40.005 158.75 0)
       (effects (font (size 1.27 1.27)) hide)
     )
@@
       (effects (font (size 1.27 1.27)) (justify right))
     )
-    (property "Footprint" "Resistor_SMD:R_0603_1608Metric_Pad0.98x0.95mm_HandSolder" (id 2) (at 40.005 167.64 0)
+    (property "Footprint" "" (id 2) (at 40.005 167.64 0)
       (effects (font (size 1.27 1.27)) hide)
     )
@@
       (effects (font (size 1.27 1.27)) (justify right))
     )
-    (property "Footprint" "Potentiometer_THT:Potentiometer_Vishay_T73XW_Horizontal" (id 2) (at 40.005 104.14 0)
+    (property "Footprint" "" (id 2) (at 40.005 104.14 0)
       (effects (font (size 1.27 1.27)) hide)
     )
@@
       (effects (font (size 1.27 1.27)) (justify left))
     )
-    (property "Footprint" "TestPoint:TestPoint_Pad_D1.5mm" (id 2) (at 59.055 93.98 0)
+    (property "Footprint" "" (id 2) (at 59.055 93.98 0)
       (effects (font (size 1.27 1.27)) hide)
     )
@@
       (effects (font (size 1.27 1.27)) (justify right))
     )
-    (property "Footprint" "Resistor_SMD:R_0603_1608Metric_Pad0.98x0.95mm_HandSolder" (id 2) (at 40.005 40.005 0)
+    (property "Footprint" "" (id 2) (at 40.005 40.005 0)
       (effects (font (size 1.27 1.27)) hide)
     )
@@
       (effects (font (size 1.27 1.27)) (justify left))
     )
-    (property "Footprint" "TestPoint:TestPoint_Pad_D1.5mm" (id 2) (at 59.055 40.005 0)
+    (property "Footprint" "" (id 2) (at 59.055 40.005 0)
       (effects (font (size 1.27 1.27)) hide)
     )
@@
       (effects (font (size 1.27 1.27)) (justify right))
     )
-    (property "Footprint" "Resistor_SMD:R_0603_1608Metric_Pad0.98x0.95mm_HandSolder" (id 2) (at 40.005 173.99 0)
+    (property "Footprint" "" (id 2) (at 40.005 173.99 0)
       (effects (font (size 1.27 1.27)) hide)
     )
@@
       (effects (font (size 1.27 1.27)) (justify right))
     )
-    (property "Footprint" "Potentiometer_THT:Potentiometer_Vishay_T73XW_Horizontal" (id 2) (at 40.005 50.165 0)
+    (property "Footprint" "" (id 2) (at 40.005 50.165 0)
       (effects (font (size 1.27 1.27)) hide)
     )
@@
       (effects (font (size 1.27 1.27)) (justify right))
     )
-    (property "Footprint" "Resistor_SMD:R_0603_1608Metric_Pad0.98x0.95mm_HandSolder" (id 2) (at 40.005 65.405 0)
+    (property "Footprint" "" (id 2) (at 40.005 65.405 0)
       (effects (font (size 1.27 1.27)) hide)
     )
@@
       (effects (font (size 1.27 1.27)) (justify left))
     )
-    (property "Footprint" "Package_TO_SOT_SMD:SOT-23" (id 2) (at 48.895 104.775 0)
+    (property "Footprint" "" (id 2) (at 48.895 104.775 0)
       (effects (font (size 1.27 1.27)) hide)
     )
@@
       (effects (font (size 1.27 1.27)) (justify right))
     )
-    (property "Footprint" "Resistor_SMD:R_0603_1608Metric_Pad0.98x0.95mm_HandSolder" (id 2) (at 40.005 113.03 0)
+    (property "Footprint" "" (id 2) (at 40.005 113.03 0)
       (effects (font (size 1.27 1.27)) hide)
     )
@@
       (effects (font (size 1.27 1.27)) (justify right))
     )
-    (property "Footprint" "Resistor_SMD:R_0603_1608Metric_Pad0.98x0.95mm_HandSolder" (id 2) (at 40.005 93.98 0)
+    (property "Footprint" "" (id 2) (at 40.005 93.98 0)
       (effects (font (size 1.27 1.27)) hide)
     )
@@
       (effects (font (size 1.27 1.27)) (justify right))
     )
-    (property "Footprint" "Resistor_SMD:R_0603_1608Metric_Pad0.98x0.95mm_HandSolder" (id 2) (at 40.005 148.59 0)
+    (property "Footprint" "" (id 2) (at 40.005 148.59 0)
       (effects (font (size 1.27 1.27)) hide)
     )
@@
       (effects (font (size 1.27 1.27)) (justify right))
     )
-    (property "Footprint" "Resistor_SMD:R_0603_1608Metric_Pad0.98x0.95mm_HandSolder" (id 2) (at 40.005 59.055 0)
+    (property "Footprint" "" (id 2) (at 40.005 59.055 0)
       (effects (font (size 1.27 1.27)) hide)
     )
@@
       (effects (font (size 1.27 1.27)) (justify left))
     )
-    (property "Footprint" "Package_TO_SOT_SMD:SOT-23" (id 2) (at 48.895 50.8 0)
+    (property "Footprint" "" (id 2) (at 48.895 50.8 0)
       (effects (font (size 1.27 1.27)) hide)
     )
@@
       (effects (font (size 1.27 1.27)) (justify left))
     )
-    (property "Footprint" "Package_TO_SOT_SMD:SOT-23" (id 2) (at 48.895 159.385 0)
+    (property "Footprint" "" (id 2) (at 48.895 159.385 0)
       (effects (font (size 1.27 1.27)) hide)
     )
@@
       (effects (font (size 1.27 1.27)) (justify left))
     )
-    (property "Footprint" "TestPoint:TestPoint_Pad_D1.5mm" (id 2) (at 59.055 148.59 0)
+    (property "Footprint" "" (id 2) (at 59.055 148.59 0)
       (effects (font (size 1.27 1.27)) hide)
     )
@@
       (effects (font (size 1.27 1.27)) (justify right))
     )
-    (property "Footprint" "Resistor_SMD:R_0603_1608Metric_Pad0.98x0.95mm_HandSolder" (id 2) (at 40.005 33.655 0)
+    (property "Footprint" "" (id 2) (at 40.005 33.655 0)
       (effects (font (size 1.27 1.27)) hide)
     )
@@
       (effects (font (size 1.27 1.27)) (justify right))
     )
-    (property "Footprint" "Resistor_SMD:R_0603_1608Metric_Pad0.98x0.95mm_HandSolder" (id 2) (at 40.005 87.63 0)
+    (property "Footprint" "" (id 2) (at 40.005 87.63 0)
       (effects (font (size 1.27 1.27)) hide)
     )
@@
       (effects (font (size 1.27 1.27)) (justify right))
     )
-    (property "Footprint" "Resistor_SMD:R_0603_1608Metric_Pad0.98x0.95mm_HandSolder" (id 2) (at 40.005 142.24 0)
-      (effects (font (size 1.27 1.27)) hide)
-    )
+    (property "Footprint" "" (id 2) (at 40.005 142.24 0)
+      (effects (font (size 1.27 1.27)) hide)
+    )

Commit message: feat(vcu): add footprint and 3D model for optocouplers
Parts:
- U4: footprint (none) -> SUFST:SOIC254P1005X380-16N
Changed lines of the file:
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@@
     (property "Reference" "U4" (id 0) (at 125.095 29.845 0))
     (property "Value" "ILQ615-4X009T" (id 1) (at 125.095 32.385 0))
-    (property "Footprint" "" (id 2) (at 125.095 46.99 0)
+    (property "Footprint" "SUFST:SOIC254P1005X380-16N" (id 2) (at 125.095 46.99 0)
       (effects (font (size 1.27 1.27)) hide)
     )

Commit message: feat(vcu): add footprints and specs for capacitors
Parts:
- D2, D3, D4, R14, R15, R16, R17, R18, R19, R2, R20, R21, R22, R23, R3, R6, R7, R8, R9, RV2, RV3, RV4, U4: Optional (none) -> False
- TP10, TP11, TP9: Optional (none) -> False; Populate True -> (none); Supplier Farnell -> (none)
Changed lines of the file:
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@@
+      (effects (font (size 1.27 1.27)) hide)
+    )
+    (property "Optional" "False" (id 4) (at 40.005 119.38 0)
       (effects (font (size 1.27 1.27)) hide)
     )
@@
     )
     (property "Datasheet" "~" (id 3) (at 40.005 158.75 0)
+      (effects (font (size 1.27 1.27)) hide)
+    )
+    (property "Optional" "False" (id 4) (at 40.005 158.75 0)
       (effects (font (size 1.27 1.27)) hide)
     )
@@
       (effects (font (size 1.27 1.27)) hide)
     )
+    (property "Optional" "False" (id 4) (at 40.005 167.64 0)
+      (effects (font (size 1.27 1.27)) hide)
+    )
     (pin "1")
     (pin "2")
@@
       (effects (font (size 1.27 1.27)) hide)
     )
+    (property "Optional" "False" (id 4) (at 40.005 104.14 0)
+      (effects (font (size 1.27 1.27)) hide)
+    )
     (pin "1")
     (pin "2")
@@
       (effects (font (size 1.27 1.27)) hide)
     )
-    (property "Supplier" "Farnell" (id 5) (at 53.975 93.98 0)
-      (effects (font (size 1.27 1.27)) hide)
-    )
-    (property "Populate" "True" (id 6) (at 53.975 93.98 0)
+    (property "Supplier" "" (id 5) (at 53.975 93.98 0)
+      (effects (font (size 1.27 1.27)) hide)
+    )
+    (property "Populate" "" (id 6) (at 53.975 93.98 0)
+      (effects (font (size 1.27 1.27)) hide)
+    )
+    (property "Optional" "False" (id 7) (at 53.975 93.98 0)
       (effects (font (size 1.27 1.27)) hide)
     )
@@
       (effects (font (size 1.27 1.27)) hide)
     )
+    (property "Optional" "False" (id 4) (at 104.775 57.15 0)
+      (effects (font (size 1.27 1.27)) hide)
+    )
     (pin "1")
     (pin "2")
@@
       (effects (font (size 1.27 1.27)) hide)
     )
+    (property "Optional" "False" (id 4) (at 40.005 40.005 0)
+      (effects (font (size 1.27 1.27)) hide)
+    )
     (pin "1")
     (pin "2")
@@
       (effects (font (size 1.27 1.27)) hide)
     )
-    (property "Supplier" "Farnell" (id 5) (at 53.975 40.005 0)
-      (effects (font (size 1.27 1.27)) hide)
-    )
-    (property "Populate" "True" (id 6) (at 53.975 40.005 0)
+    (property "Supplier" "" (id 5) (at 53.975 40.005 0)
+      (effects (font (size 1.27 1.27)) hide)
+    )
+    (property "Populate" "" (id 6) (at 53.975 40.005 0)
+      (effects (font (size 1.27 1.27)) hide)
+    )
+    (property "Optional" "False" (id 7) (at 53.975 40.005 0)
       (effects (font (size 1.27 1.27)) hide)
     )
@@
       (effects (font (size 1.27 1.27)) hide)
     )
+    (property "Optional" "False" (id 4) (at 40.005 173.99 0)
+      (effects (font (size 1.27 1.27)) hide)
+    )
     (pin "1")
     (pin "2")
@@
       (effects (font (size 1.27 1.27)) hide)
     )
+    (property "Optional" "False" (id 4) (at 40.005 50.165 0)
+      (effects (font (size 1.27 1.27)) hide)
+    )
     (pin "1")
     (pin "2")
@@
       (effects (font (size 1.27 1.27)) hide)
     )
+    (property "Optional" "False" (id 4) (at 40.005 65.405 0)
+      (effects (font (size 1.27 1.27)) hide)
+    )
     (pin "1")
     (pin "2")
@@
       (effects (font (size 1.27 1.27)) hide)
     )
+    (property "Optional" "False" (id 4) (at 48.895 104.775 0)
+      (effects (font (size 1.27 1.27)) hide)
+    )
     (pin "1")
     (pin "2")
@@
       (effects (font (size 1.27 1.27)) hide)
     )
+    (property "Optional" "False" (id 4) (at 40.005 113.03 0)
+      (effects (font (size 1.27 1.27)) hide)
+    )
     (pin "1")
     (pin "2")
@@
       (effects (font (size 1.27 1.27)) hide)
     )
+    (property "Optional" "False" (id 4) (at 40.005 93.98 0)
+      (effects (font (size 1.27 1.27)) hide)
+    )
     (pin "1")
     (pin "2")
@@
     )
     (property "Datasheet" "~" (id 3) (at 40.005 148.59 0)
+      (effects (font (size 1.27 1.27)) hide)
+    )
+    (property "Optional" "False" (id 4) (at 40.005 148.59 0)
       (effects (font (size 1.27 1.27)) hide)
     )
@@
       (effects (font (size 1.27 1.27)) hide)
     )
+    (property "Optional" "False" (id 4) (at 104.775 67.31 0)
+      (effects (font (size 1.27 1.27)) hide)
+    )
     (pin "1")
     (pin "2")
@@
     )
     (property "Datasheet" "~" (id 3) (at 40.005 59.055 0)
+      (effects (font (size 1.27 1.27)) hide)
+    )
+    (property "Optional" "False" (id 4) (at 40.005 59.055 0)
       (effects (font (size 1.27 1.27)) hide)
     )
@@
       (effects (font (size 1.27 1.27)) hide)
     )
+    (property "Optional" "False" (id 4) (at 104.775 36.83 0)
+      (effects (font (size 1.27 1.27)) hide)
+    )
     (pin "1")
     (pin "2")
@@
     )
     (property "Datasheet" "https://diotec.com/tl_files/diotec/files/pdf/datasheets/bzx84c2v4.pdf" (id 3) (at 48.895 50.8 0)
+      (effects (font (size 1.27 1.27)) hide)
+    )
+    (property "Optional" "False" (id 4) (at 48.895 50.8 0)
       (effects (font (size 1.27 1.27)) hide)
     )
@@
     )
     (property "Order Code" "782-ILQ615-4X009" (id 5) (at 125.095 46.99 0)
+      (effects (font (size 1.27 1.27)) hide)
+    )
+    (property "Optional" "False" (id 6) (at 125.095 46.99 0)
       (effects (font (size 1.27 1.27)) hide)
     )
@@
       (effects (font (size 1.27 1.27)) hide)
     )
+    (property "Optional" "False" (id 4) (at 48.895 159.385 0)
+      (effects (font (size 1.27 1.27)) hide)
+    )
     (pin "1")
     (pin "2")
@@
       (effects (font (size 1.27 1.27)) hide)
     )
-    (property "Supplier" "Farnell" (id 5) (at 53.975 148.59 0)
-      (effects (font (size 1.27 1.27)) hide)
-    )
-    (property "Populate" "True" (id 6) (at 53.975 148.59 0)
+    (property "Supplier" "" (id 5) (at 53.975 148.59 0)
+      (effects (font (size 1.27 1.27)) hide)
+    )
+    (property "Populate" "" (id 6) (at 53.975 148.59 0)
+      (effects (font (size 1.27 1.27)) hide)
+    )
+    (property "Optional" "False" (id 7) (at 53.975 148.59 0)
       (effects (font (size 1.27 1.27)) hide)
     )
@@
     )
     (property "Datasheet" "~" (id 3) (at 40.005 33.655 0)
+      (effects (font (size 1.27 1.27)) hide)
+    )
+    (property "Optional" "False" (id 4) (at 40.005 33.655 0)
       (effects (font (size 1.27 1.27)) hide)
     )
@@
     )
     (property "Datasheet" "~" (id 3) (at 40.005 87.63 0)
+      (effects (font (size 1.27 1.27)) hide)
+    )
+    (property "Optional" "False" (id 4) (at 40.005 87.63 0)
       (effects (font (size 1.27 1.27)) hide)
     )
@@
       (effects (font (size 1.27 1.27)) hide)
     )
+    (property "Optional" "False" (id 4) (at 104.775 46.99 0)
+      (effects (font (size 1.27 1.27)) hide)
+    )
     (pin "1")
     (pin "2")
@@
       (effects (font (size 1.27 1.27)) hide)
     )
+    (property "Optional" "False" (id 4) (at 40.005 142.24 0)
+      (effects (font (size 1.27 1.27)) hide)
+    )

Commit message: feat(vcu): add footprints for zener diodes
Parts:
- D2, D3, D4: value 3V3 -> BZX84-C3V3; Order Code (none) -> 771-BZX84-C3V3-T/R; Supplier (none) -> Mouser
Changed lines of the file:
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@@
       (effects (font (size 1.27 1.27)) (justify left))
     )
-    (property "Value" "3V3" (id 1) (at 51.435 106.045 90)
+    (property "Value" "BZX84-C3V3" (id 1) (at 51.435 106.045 90)
       (effects (font (size 1.27 1.27)) (justify left))
     )
@@
       (effects (font (size 1.27 1.27)) hide)
     )
-    (property "Datasheet" "https://diotec.com/tl_files/diotec/files/pdf/datasheets/bzx84c2v4.pdf" (id 3) (at 48.895 104.775 0)
+    (property "Datasheet" "https://www.mouser.co.uk/datasheet/2/916/BZX84_SER-1319896.pdf" (id 3) (at 48.895 104.775 0)
       (effects (font (size 1.27 1.27)) hide)
     )
     (property "Optional" "False" (id 4) (at 48.895 104.775 0)
+      (effects (font (size 1.27 1.27)) hide)
+    )
+    (property "Order Code" "771-BZX84-C3V3-T/R" (id 5) (at 48.895 104.775 0)
+      (effects (font (size 1.27 1.27)) hide)
+    )
+    (property "Supplier" "Mouser" (id 6) (at 48.895 104.775 0)
       (effects (font (size 1.27 1.27)) hide)
     )
@@
       (effects (font (size 1.27 1.27)) (justify left))
     )
-    (property "Value" "3V3" (id 1) (at 51.435 52.07 90)
+    (property "Value" "BZX84-C3V3" (id 1) (at 51.435 52.07 90)
       (effects (font (size 1.27 1.27)) (justify left))
     )
@@
       (effects (font (size 1.27 1.27)) hide)
     )
-    (property "Datasheet" "https://diotec.com/tl_files/diotec/files/pdf/datasheets/bzx84c2v4.pdf" (id 3) (at 48.895 50.8 0)
+    (property "Datasheet" "https://www.mouser.co.uk/datasheet/2/916/BZX84_SER-1319896.pdf" (id 3) (at 48.895 50.8 0)
       (effects (font (size 1.27 1.27)) hide)
     )
     (property "Optional" "False" (id 4) (at 48.895 50.8 0)
+      (effects (font (size 1.27 1.27)) hide)
+    )
+    (property "Order Code" "771-BZX84-C3V3-T/R" (id 5) (at 48.895 50.8 0)
+      (effects (font (size 1.27 1.27)) hide)
+    )
+    (property "Supplier" "Mouser" (id 6) (at 48.895 50.8 0)
       (effects (font (size 1.27 1.27)) hide)
     )
@@
       (effects (font (size 1.27 1.27)) (justify left))
     )
-    (property "Value" "3V3" (id 1) (at 50.8 160.655 90)
+    (property "Value" "BZX84-C3V3" (id 1) (at 50.8 160.655 90)
       (effects (font (size 1.27 1.27)) (justify left))
     )
@@
       (effects (font (size 1.27 1.27)) hide)
     )
-    (property "Datasheet" "https://diotec.com/tl_files/diotec/files/pdf/datasheets/bzx84c2v4.pdf" (id 3) (at 48.895 159.385 0)
+    (property "Datasheet" "https://www.mouser.co.uk/datasheet/2/916/BZX84_SER-1319896.pdf" (id 3) (at 48.895 159.385 0)
       (effects (font (size 1.27 1.27)) hide)
     )
@@
       (effects (font (size 1.27 1.27)) hide)
     )
+    (property "Order Code" "771-BZX84-C3V3-T/R" (id 5) (at 48.895 159.385 0)
+      (effects (font (size 1.27 1.27)) hide)
+    )
+    (property "Supplier" "Mouser" (id 6) (at 48.895 159.385 0)
+      (effects (font (size 1.27 1.27)) hide)
+    )
