File: vcu/vcu_docs.kicad_sch (KiCad schematic)
At the start: 0 parts

Commit message: schematic notes
Other:
- company: (none) -> SUFST
- title: (none) -> Vehicle Control Unit
Changed lines of the file:
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@@
 	(generator_version "9.0")
 	(paper "A4")
+	(title_block
+		(title "Vehicle Control Unit")
+		(date "2026-01-05")
+		(rev "1")
+		(company "SUFST")
+		(comment 1 "Annabel Owen")
+	)
 	(text "debug header explanation\n- board ideas\n- reverse prot\n\nprogramming options\n\nsd card\n-sd card button\n\nusb vs glv power\n- power mux situation\n- ldo \n- analog filter\n\neeprom and temp sensor\n\nimu\n- swappable with footprint\n- extra bus hooked up\n\nnet naming conventions for power\n\nadc\n- sims\n- theory\n- why ive done it\n- screenshot examples of hookup\n- justify amp choice \n- dnfs\n- voltage divider\n- over voltage prot\n- design principle\n- analog vs spice filter designer\n\ncan overveiw\n"
 		(exclude_from_sim no)

Commit message: silkscreen additions
Other:
- note removed: "debug header explanation - board ideas - reverse prot programming options sd card -sd card button usb vs glv power - power mux situation - ldo - analog filter eeprom and temp sensor imu - swappable with footprint - extra bus hooked up net naming conventions for power adc - sims - theory - why ive done it - screenshot examples of hookup - justify amp choice - dnfs - voltage divider - over voltage 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"
- note removed: "peripheral table: - each perhiferal - colour code - pins for each - description of use - stm name leave adc docs in adc file high side explanation - how levle shifter works - how star works - high speed vs low speed inputs - led outs - how latch works - how check works - how rtd works - pwm outputs - tvs option overall pcb design principle explanation list of useful app notes with references powe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"
Changed lines of the file:
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@@
 		(rev "1")
 		(company "SUFST")
-		(comment 1 "Annabel Owen")
-	)
-	(text "debug header explanation\n- board ideas\n- reverse prot\n\nprogramming options\n\nsd card\n-sd card button\n\nusb vs glv power\n- power mux situation\n- ldo \n- analog filter\n\neeprom and temp sensor\n\nimu\n- swappable with footprint\n- extra bus hooked up\n\nnet naming conventions for power\n\nadc\n- sims\n- theory\n- why ive done it\n- screenshot examples of hookup\n- justify amp choice \n- dnfs\n- voltage divider\n- over voltage prot\n- design principle\n- analog vs spice filter designer\n\ncan overveiw\n"
-		(exclude_from_sim no)
-		(at 96.774 54.356 0)
-		(effects
-			(font
-				(size 1.27 1.27)
-				(thickness 0.1588)
-			)
-			(justify left)
-		)
-	)
-	(text "peripheral table:\n- each perhiferal\n- colour code\n- pins for each\n- description of use\n- stm name\n\nleave adc docs in adc file\n\nhigh side explanation\n- how levle shifter works\n- how star works\n- high speed vs low speed inputs\n- led outs\n- how latch works\n- how check works\n- how rtd works\n- pwm outputs\n- tvs option\n\noverall pcb design principle explanation\n\nlist of useful app notes with references\n\npower stage explanation and limits\n"
-		(exclude_from_sim no)
-		(at 37.084 44.45 0)
-		(effects
-			(font
-				(size 1.27 1.27)
-			)
-			(justify left)
-		)
+		(comment 1 "cannabel")
 	)
 )

Commit message: Design review changes
Other:
- title: Vehicle Control Unit -> Vehicle Control Unit Test
Changed lines of the file:
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@@
 	(paper "A4")
 	(title_block
-		(title "Vehicle Control Unit")
-		(date "2026-01-05")
-		(rev "1")
+		(title "Vehicle Control Unit Test")
+		(date "2026-02-01")
+		(rev "v3.0.0")
 		(company "SUFST")
-		(comment 1 "cannabel")
+		(comment 1 "STAG 12")
+		(comment 2 "Annabel Owen")
+		(comment 3 "Adam Eastman, Ray Wang, John McGarvey")
+		(comment 4 "26-E99-001-0")
 	)
 )
