File: precharge/hv.kicad_sch (KiCad schematic)
At the start: 51 parts, among them Q1 BC856, Q2 BC856, Q3 BC856, U4 TLV274

Commit message: chore(all) renamed BSPD files to remove version number from name, moved all symbols from individual symbol libraries into common/sufts-lib.kicad_sym, combined all project specific footprint folders into common/sufts-lib.pretty, moved all project specific step files into common/step, fixed all paths making them relative, fixed all broken cad models on pcbs. missing one cad model that is simply impossible to find online. imported discharge relay breakout pcb folder.
Parts:
- F1: footprint footprints:fuseholder -> SUFST:fuseholder
Changed lines of the file:
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@@
     (property "Reference" "F1" (id 0) (at 171.45 95.6015 90))
     (property "Value" "Fuse" (id 1) (at 171.45 98.3766 90))
-    (property "Footprint" "footprints:fuseholder" (id 2) (at 171.45 102.108 90)
+    (property "Footprint" "SUFST:fuseholder" (id 2) (at 171.45 102.108 90)
       (effects (font (size 1.27 1.27)) hide)
     )
