File: precharge/relays.kicad_sch (KiCad schematic)
At the start: 11 parts, among them K1 G5Q-1A-EU DC12, K2 G5Q-1A-EU DC12, Q1 XP262N7002TR-G, Q2 XP262N7002TR-G, Q3 XP262N7002TR-G, Q4 XP262N7002TR-G, Q5 XP262N7002TR-G

Commit message: feat(precharge): first draft of new layout
Parts:
- K1, K2: footprint SUFST:PCH-112L2MH -> SUFST:Relay_SPDT_Omron-G5Q-1
- NT2: footprint (none) -> NetTie:NetTie-2_SMD_Pad0.5mm

Commit message: fix(precharge): fixed some issues after review
Parts:
- removed D4: SS14+, Diode_SMD:D_SMA, symbol Device:D
Other:
- note added: "Relay has diode built in"
Changed lines of the file:
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@@
     (effects (font (size 1.27 1.27)) (justify left bottom))
+  )
+  (text "Relay has diode built in" (at 186.055 128.27 0)
+    (effects (font (size 1.27 1.27)) (justify right bottom))
   )
   (text "Only power pre-charge\nrelay if -ve AIR is\npowered (shutdown \nloop closed)"
@@
         )
       )
-    )
-  )
-  (symbol (lib_id "Device:D") (at 144.78 128.27 270) (unit 1)
-    (in_bom yes) (on_board yes) (dnp no)
-    (property "Reference" "D4" (at 140.97 125.095 90)
-      (effects (font (size 1.27 1.27)) (justify left))
-    )
-    (property "Value" "SS14+" (at 138.43 131.445 90)
-      (effects (font (size 1.27 1.27)) (justify left))
-    )
-    (property "Footprint" "Diode_SMD:D_SMA" (at 144.78 128.27 0)
-      (effects (font (size 1.27 1.27)) hide)
-    )
-    (property "Datasheet" "~" (at 144.78 128.27 0)
-      (effects (font (size 1.27 1.27)) hide)
-    )
-    (pin "1")
-    (pin "2")
-    (instances
-      (project "precharge"
-        (path "/5e0e9869-af81-4a3e-ad08-271d45318b88/69e1a8e2-aecd-4790-9267-94ebdba414d7"
-          (reference "D4") (unit 1)
-        )
-      )

Commit message: feat(precharge): update sheet info and docs
Other:
- company: (none) -> SUFST - Southampton University Formula Student Team
- title: (none) -> Pre-Charge
Changed lines of the file:
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@@
 (kicad_sch (version 20230121) (generator eeschema)
   (paper "A4")
+  (title_block
+    (title "Pre-Charge")
+    (date "2023-04-27")
+    (rev "2.0.0")
+    (company "SUFST - Southampton University Formula Student Team")
+    (comment 1 "STAG 9")
+    (comment 2 "Tim Brewis")
+    (comment 3 "Max O'Brien, Marek Frodyma")
+  )
   (junction (at 88.9 80.01) (diameter 0) (color 0 0 0 0)
   )
   (junction (at 109.22 80.01) (diameter 0) (color 0 0 0 0)
-  )
-  (junction (at 149.86 121.92) (diameter 0) (color 0 0 0 0)
   )
   (junction (at 154.94 59.69) (diameter 0) (color 0 0 0 0)
@@
   )
   (junction (at 123.19 109.22) (diameter 0) (color 0 0 0 0)
-  )
-  (junction (at 149.86 134.62) (diameter 0) (color 0 0 0 0)
   )
   (junction (at 149.86 59.69) (diameter 0) (color 0 0 0 0)
@@
     (stroke (width 0) (type default))
   )
-  (wire (pts (xy 144.78 124.46) (xy 144.78 121.92))
-    (stroke (width 0) (type default))
-  )
   (wire (pts (xy 77.47 109.22) (xy 123.19 109.22))
     (stroke (width 0) (type default))
@@
   )
   (wire (pts (xy 180.34 72.39) (xy 177.8 72.39))
-    (stroke (width 0) (type default))
-  )
-  (wire (pts (xy 144.78 134.62) (xy 149.86 134.62))
     (stroke (width 0) (type default))
   )
@@
     (stroke (width 0) (type default))
   )
-  (wire (pts (xy 144.78 121.92) (xy 149.86 121.92))
-    (stroke (width 0) (type default))
-  )
   (wire (pts (xy 88.9 69.85) (xy 91.44 69.85))
     (stroke (width 0) (type default))
@@
     (stroke (width 0) (type default))
   )
-  (wire (pts (xy 144.78 132.08) (xy 144.78 134.62))
-    (stroke (width 0) (type default))
-  )
