File: lvbms-relay/relay/relay.kicad_sch (KiCad schematic)
At the start: 5 parts, among them Q2 XP262N7002TR-G

Commit message: Full BMS Schematic Draft 1
Connections:
- net GND: no longer U1.COM
- net VDD: now also D2.3 (K); no longer D2.1 (A)
- net at Q2.3 (D), U1.C1 (COIL1): now also D2.1 (A); no longer D2.3 (K)
Other:
- moved on the sheet: D2
Changed lines of the file:
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@@
   (junction (at 166.37 130.81) (diameter 0) (color 0 0 0 0)
   )
-  (wire (pts (xy 176.53 99.06) (xy 177.8 99.06))
-    (stroke (width 0) (type default))
-  )
   (wire (pts (xy 166.37 97.79) (xy 166.37 102.87))
     (stroke (width 0) (type default))
   )
+  (wire (pts (xy 153.67 88.9) (xy 153.67 77.47))
+    (stroke (width 0) (type default))
+  )
+  (wire (pts (xy 179.07 77.47) (xy 179.07 82.55))
+    (stroke (width 0) (type default))
+  )
+  (wire (pts (xy 154.94 130.81) (xy 154.94 118.11))
+    (stroke (width 0) (type default))
+  )
+  (wire (pts (xy 149.86 118.11) (xy 154.94 118.11))
+    (stroke (width 0) (type default))
+  )
+  (wire (pts (xy 154.94 130.81) (xy 157.48 130.81))
+    (stroke (width 0) (type default))
+  )
+  (wire (pts (xy 153.67 96.52) (xy 153.67 102.87))
+    (stroke (width 0) (type default))
+  )
+  (wire (pts (xy 179.07 77.47) (xy 189.23 77.47))
+    (stroke (width 0) (type default))
+  )
+  (wire (pts (xy 166.37 123.19) (xy 166.37 130.81))
+    (stroke (width 0) (type default))
+  )
   (wire (pts (xy 166.37 68.58) (xy 166.37 77.47))
     (stroke (width 0) (type default))
   )
-  (wire (pts (xy 177.8 99.06) (xy 177.8 104.14))
-    (stroke (width 0) (type default))
-  )
-  (wire (pts (xy 154.94 88.9) (xy 154.94 77.47))
-    (stroke (width 0) (type default))
-  )
-  (wire (pts (xy 179.07 77.47) (xy 179.07 82.55))
-    (stroke (width 0) (type default))
-  )
-  (wire (pts (xy 154.94 130.81) (xy 154.94 118.11))
-    (stroke (width 0) (type default))
-  )
-  (wire (pts (xy 149.86 118.11) (xy 154.94 118.11))
-    (stroke (width 0) (type default))
-  )
-  (wire (pts (xy 154.94 130.81) (xy 157.48 130.81))
-    (stroke (width 0) (type default))
-  )
-  (wire (pts (xy 154.94 96.52) (xy 154.94 102.87))
-    (stroke (width 0) (type default))
-  )
-  (wire (pts (xy 179.07 77.47) (xy 189.23 77.47))
-    (stroke (width 0) (type default))
-  )
-  (wire (pts (xy 166.37 123.19) (xy 166.37 130.81))
-    (stroke (width 0) (type default))
-  )
   (wire (pts (xy 154.94 118.11) (xy 158.75 118.11))
     (stroke (width 0) (type default))
   )
-  (wire (pts (xy 154.94 102.87) (xy 166.37 102.87))
-    (stroke (width 0) (type default))
-  )
-  (wire (pts (xy 176.53 97.79) (xy 176.53 99.06))
+  (wire (pts (xy 153.67 102.87) (xy 166.37 102.87))
     (stroke (width 0) (type default))
   )
@@
     (stroke (width 0) (type default))
   )
-  (wire (pts (xy 154.94 77.47) (xy 166.37 77.47))
+  (wire (pts (xy 153.67 77.47) (xy 166.37 77.47))
     (stroke (width 0) (type default))
   )
@@
       (effects (font (size 1.27 1.27)) hide)
     )
+    (pin "1")
     (pin "2")
-    (pin "1")
     (instances
       (project "relay"
@@
     )
   )
-  (symbol (lib_id "Diode:BAT54W") (at 154.94 92.71 270) (mirror x) (unit 1)
+  (symbol (lib_id "Diode:BAT54W") (at 153.67 92.71 90) (mirror x) (unit 1)
     (in_bom yes) (on_board yes) (dnp no)
-    (property "Reference" "D2" (at 149.86 92.71 0)
-      (effects (font (size 1.27 1.27)))
-    )
-    (property "Value" "BAT54W" (at 151.765 92.075 0)
-      (effects (font (size 1.27 1.27)))
-    )
-    (property "Footprint" "Package_TO_SOT_SMD:SOT-323_SC-70" (at 150.495 92.71 0)
-      (effects (font (size 1.27 1.27)) hide)
-    )
-    (property "Datasheet" "https://assets.nexperia.com/documents/data-sheet/BAT54W_SER.pdf" (at 154.94 92.71 0)
-      (effects (font (size 1.27 1.27)) hide)
-    )
-    (property "Supplier" "Mouser" (at 154.94 92.71 0)
-      (effects (font (size 1.27 1.27)) hide)
-    )
-    (property "Order Code" "771-BAT54W-T/R" (at 154.94 92.71 0)
+    (property "Reference" "D2" (at 158.75 92.71 0)
+      (effects (font (size 1.27 1.27)))
+    )
+    (property "Value" "BAT54W" (at 156.845 93.345 0)
+      (effects (font (size 1.27 1.27)))
+    )
+    (property "Footprint" "Package_TO_SOT_SMD:SOT-323_SC-70" (at 158.115 92.71 0)
+      (effects (font (size 1.27 1.27)) hide)
+    )
+    (property "Datasheet" "https://assets.nexperia.com/documents/data-sheet/BAT54W_SER.pdf" (at 153.67 92.71 0)
+      (effects (font (size 1.27 1.27)) hide)
+    )
+    (property "Supplier" "Mouser" (at 153.67 92.71 0)
+      (effects (font (size 1.27 1.27)) hide)
+    )
+    (property "Order Code" "771-BAT54W-T/R" (at 153.67 92.71 0)
       (effects (font (size 1.27 1.27)) hide)
     )
@@
       (effects (font (size 1.27 1.27)) hide)
     )
+    (pin "1")
     (pin "2")
-    (pin "1")
     (instances
       (project "relay"
         (path "/36d30ecc-cf8c-4837-baa1-a7465520d969"
           (reference "R2") (unit 1)
-        )
-      )
-    )
-  )
-  (symbol (lib_id "power:GND") (at 177.8 104.14 0) (unit 1)
-    (in_bom yes) (on_board yes) (dnp no) (fields_autoplaced)
-    (property "Reference" "#PWR02" (at 177.8 110.49 0)
-      (effects (font (size 1.27 1.27)) hide)
-    )
-    (property "Value" "GND" (at 177.8 109.22 0)
-      (effects (font (size 1.27 1.27)))
-    )
-    (property "Footprint" "" (at 177.8 104.14 0)
-      (effects (font (size 1.27 1.27)) hide)
-    )
-    (property "Datasheet" "" (at 177.8 104.14 0)
-      (effects (font (size 1.27 1.27)) hide)
-    )
-    (pin "1")
-    (instances
-      (project "relay"
-        (path "/36d30ecc-cf8c-4837-baa1-a7465520d969"
-          (reference "#PWR02") (unit 1)
         )
       )
@@
     (pin "C1")
     (pin "C2")
+    (pin "COM")
     (pin "NO")
-    (pin "COM")
-    (instances
-      (project "relay"
+    (instances
+      (project "relay"
