File: ail-LED/ail-LED_handsolder.kicad_sch (KiCad schematic)
At the start: 20 parts, among them J1 LED, Q1 BC817

Commit message: Revised PCB to support hand soldering
Parts:
- D1, D10, D11, D12, D2, D3, D4, D5, D6, D7, D8, D9: footprint SUFST:KR-SITQA1.23_reflow -> SUFST:KR-SITQA1.23_handsolder
- J1: symbol Connector_Generic:Conn_01x02 -> Connector_Generic:Conn_01x04
Connections:
- net LED-: now reaches D12.1 (K), Q1.3 (C)
- net Input: now reaches D1.2 (A), J1.2 (Pin_2), R1.1
- net REG: now reaches D13.1 (K), Q1.1 (B), R1.2
- net GND: now reaches D13.2 (A), J1.1 (Pin_1), R2.2, RV1.2
- net TRIM: now reaches Q1.2 (E), R2.1, RV1.3
- new net MOUNT: J1.3 (Pin_3), J1.4 (Pin_4)
