File: lvbms/BatteryBalancing.kicad_sch (KiCad schematic)
At the start: 15 parts, among them Q1 BC807, Q2 BC807, Q3 BC807, Q4 BC817, Q5 BC817, Q6 BC817

Commit message: Various adjustments
Connections:
- net at Q2.1 (B): now also R28.2; no longer R28.1
- net at Q4.3 (C): now also R27.1; no longer R27.2
- net at Q3.1 (B): now also R29.2; no longer R29.1
- net at Q6.3 (C): now also R29.1; no longer R29.2
- net at Q5.3 (C): now also R28.1; no longer R28.2
- net at Q1.1 (B): now also R27.2; no longer R27.1
Other:
- note added: "BJT leakage current ~100nA when off. Will drain 1Ah in ~100 years."
- moved on the sheet: Q1, Q2, Q3, Q4, Q5, Q6, R24, R25, R26, R27, R28, R29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

Commit message: Added order codes for most components
Parts:
- Q1, Q2, Q3: Order Code (none) -> 637-BC807-25; Supplier (none) -> Mouser
- Q4, Q5, Q6: Order Code (none) -> 637-BC817-40-Q; Supplier (none) -> Mouser
Changed lines of the file:
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@@
       (effects (font (size 1.27 1.27)) (justify left) hide)
+    )
+    (property "Order Code" "637-BC807-25" (at 97.155 84.455 0)
+      (effects (font (size 1.27 1.27)) hide)
+    )
+    (property "Supplier" "Mouser" (at 97.155 84.455 0)
+      (effects (font (size 1.27 1.27)) hide)
     )
     (pin "1")
@@
       (effects (font (size 1.27 1.27)) (justify left) hide)
     )
+    (property "Order Code" "637-BC817-40-Q" (at 113.03 59.055 0)
+      (effects (font (size 1.27 1.27)) hide)
+    )
+    (property "Supplier" "Mouser" (at 113.03 59.055 0)
+      (effects (font (size 1.27 1.27)) hide)
+    )
     (pin "1")
     (pin "2")
@@
       (effects (font (size 1.27 1.27)) (justify left) hide)
     )
+    (property "Order Code" "637-BC807-25" (at 97.155 128.905 0)
+      (effects (font (size 1.27 1.27)) hide)
+    )
+    (property "Supplier" "Mouser" (at 97.155 128.905 0)
+      (effects (font (size 1.27 1.27)) hide)
+    )
     (pin "1")
     (pin "2")
@@
       (effects (font (size 1.27 1.27)) (justify left) hide)
     )
+    (property "Order Code" "637-BC807-25" (at 97.155 37.465 0)
+      (effects (font (size 1.27 1.27)) hide)
+    )
+    (property "Supplier" "Mouser" (at 97.155 37.465 0)
+      (effects (font (size 1.27 1.27)) hide)
+    )
     (pin "1")
     (pin "2")
@@
       (effects (font (size 1.27 1.27)) (justify left) hide)
     )
+    (property "Order Code" "637-BC817-40-Q" (at 113.03 155.575 0)
+      (effects (font (size 1.27 1.27)) hide)
+    )
+    (property "Supplier" "Mouser" (at 113.03 155.575 0)
+      (effects (font (size 1.27 1.27)) hide)
+    )
     (pin "1")
     (pin "2")
@@
       (effects (font (size 1.27 1.27)) (justify left) hide)
     )
-    (pin "1")
+    (property "Order Code" "637-BC817-40-Q" (at 113.03 104.775 0)
+      (effects (font (size 1.27 1.27)) hide)
+    )
+    (property "Supplier" "Mouser" (at 113.03 104.775 0)
+      (effects (font (size 1.27 1.27)) hide)
+    )
+    (pin "1")
