File: gps/GPS Schematic/GPS_Schematic_main/untitled2.kicad_sch (KiCad schematic)
At the start: 30 parts, among them IC1 TCAN3404DRQ1, IC4 TLV1117LV33DCYR, IC5 MAX3232ECWE+, J3 UJ20-C-H-G-SMT-5-P16-TR, Q1 140107146000, U3 SMTU2032-LF

Commit message: Done mostly all of design for schematic
Hello everybody my name is markiplier,
need to add connectors to schematic
**IGNORE GPS PCB IT IS OUTDATED**
Parts:
- removed C16, C17: 10uF, Capacitor_SMD:C_0805_2012Metric, symbol PCM_Capacitor_US_AKL:C_Generic
- removed F1: 0ZCH0050FF2G, Fuse:Fuse_1210_3225Metric_Pad1.42x2.65mm_HandSolder, symbol Device:Polyfuse
- removed IC4: TLV1117LV33DCYR, Sufst_GPS:SOT230P700X180-4N, symbol TLV1117LV33DCYR:TLV1117LV33DCYR
- removed JP3: FUSE BYPASS, Jumper:SolderJumper-2_P1.3mm_Open_RoundedPad1.0x1.5mm, symbol Jumper:SolderJumper_2_Open
- added J5: Conn_02x05_Odd_Even, symbol Connector_Generic:Conn_02x05_Odd_Even
Connections:
- net +3.3V: now also J5.1 (Pin_1)
- net GND: now also J5.9 (Pin_9)
- net GPS_RX renamed GPS1_RX
- net GPS_TX renamed GPS1_TX
- new net EXT_RADIO_0: J5.8 (Pin_8)
- new net EXT_RADIO_1: J5.10 (Pin_10)
- new net EXT_RADIO_CS: J5.6 (Pin_6)
- new net GPS2_RX: J5.2 (Pin_2)
- new net GPS2_TX: J5.4 (Pin_4)
- new net SPI1_MISO: J5.5 (Pin_5)
- new net SPI1_MOSI: J5.3 (Pin_3)
- new net SPI1_SCK: J5.7 (Pin_7)
Other:
- note added: "According to all known laws of aviation, there is no way a bee should be able to fly. Its wings are too small to get its fat little body off the ground. The bee, of course, flies anyway because bees don't care what humans think is impossible."
- note added: "External Radio header for RTK Functionality, can attach another mcu to directly feed into gps using gps usart 2 pins"
- note added: "Lap timer outputs using TTL voltage levels, this makes it so it dont fry it, pins should be connected with internal pullup"
- note added: "Radio Header"
- note added: "USB connected to GPS chip for ublox config, should be routed with differential pairing for usb HS"
- note added: "used for GPS hot start and maybe mcu things??, important tho"
- note added: "used to connect and communicate with the logger, cx and cts pins added if logger changes and it needs it"
- note removed: "5v to 3.3v LDO"
- company: (none) -> Sheet - Alex. L
- title: EXT Pheripheral + Power -> EXT Pheripheral chips + LDO
- moved on the sheet: U3
