File: gps/GPS Schematic/GPS_Schematic_main/GPS_GPSndPOWER.kicad_sch (KiCad schematic)
At the start: 31 parts, among them IC6 TLV75901PDRVT, J6 LOGGER_CONN, J7 PWR_CONN, J8 LAP_TIMER, J9 73251-2200, U2 ZED-F9P, U4 LMR336300CDDA

Commit message: Finished Everything Hopefully
Mama Mia!
Parts:
- removed D8: S2JTR, Diode_SMD:D_SMB, symbol Diode:S2JTR
- removed J6: LOGGER_CONN, symbol Connector_Generic:Conn_02x04_Odd_Even
- removed J7: PWR_CONN, symbol Connector_Generic:Conn_02x04_Odd_Even
- removed J8: LAP_TIMER, symbol Connector_Generic:Conn_02x02_Odd_Even
- added GPS_RESET1: SolderJumper_2_Open, Jumper:SolderJumper-2_P1.3mm_Open_RoundedPad1.0x1.5mm, symbol Jumper:SolderJumper_2_Open
- added J6: Conn_02x06_Odd_Even, Connector_Molex:Molex_Micro-Fit_3.0_43045-1200_2x06_P3.00mm_Horizontal, symbol Connector_Generic:Conn_02x06_Odd_Even
- added R17: 10k, PCM_Resistor_SMD_AKL:R_0805_2012Metric, symbol Device:R
- added R18: 90k, PCM_Resistor_SMD_AKL:R_0805_2012Metric, symbol Device:R
- added TP5, TP6, TP7: TestPoint, TestPoint:TestPoint_Pad_D1.5mm, symbol Connector:TestPoint
- added U5: TPS2116DRL, Package_TO_SOT_SMD:SOT-583-8, symbol Power_Management:TPS2116DRL
- C30: footprint Capacitor_SMD:C_0603_1608Metric -> Capacitor_SMD:C_0805_2012Metric
- C31, C32, C33: footprint Capacitor_SMD:C_0402_1005Metric -> Capacitor_SMD:C_0805_2012Metric
- J9: footprint (none) -> Sufst_GPS:73251-2200
- R13, R14: footprint Resistor_SMD:R_0402_1005Metric -> PCM_Resistor_SMD_AKL:R_0805_2012Metric
Connections:
- net +12V: now also J6.1 (Pin_1)
- net +3.3V: now also TP6.1
- net +5V: now also TP7.1, U5.2 (VOUT), U5.7 (VOUT)
- net CAN_H: now also J6.3 (Pin_3), J6.4 (Pin_4)
- net CAN_L: now also J6.5 (Pin_5), J6.6 (Pin_6)
- net GND: now also GPS_RESET1.1 (A), J6.12 (Pin_12), J6.2 (Pin_2), R18.1, U5.1 (GND)
- net GPS_NRST: now also GPS_RESET1.2 (B)
- net LAP_TIMER_IN: now also J6.11 (Pin_11)
- net RS232_CTS: now also J6.10 (Pin_10)
- net RS232_CX: now also J6.9 (Pin_9)
- net RS232_RX: now also J6.7 (Pin_7)
- net RS232_TX: now also J6.8 (Pin_8)
- net +5V StepDown: now reaches C34.1, C35.1, L1.2, R13.2
- net +5V StepDown: now also R17.2, TP5.1, U5.3 (VIN1), U5.5 (MODE)
- net USB_DM renamed USB_DN
- new net: R17.1, R18.2, U5.4 (PR1)
- new net +5V USB: U5.6 (VIN2)
- no-connect marks 9 -> 10
Other:
- note removed: "This is only a stand in for the connectors because idk what to use and no one is really helpful"
- moved on the sheet: GPS_UPDATE1
