File: gps/GPS Schematic/GPS_Schematic_main/GPS_PERHIPHERALS.kicad_sch (KiCad schematic)
At the start: 26 parts, among them IC1 TCAN3404DRQ1, IC5 MAX3232ECWE+, J3 UJ20-C-H-G-SMT-5-P16-TR, J5 Conn_02x05_Odd_Even, Q1 140107146000, U3 SMTU2032-LF

Commit message: Finished Everything Hopefully
Mama Mia!
Parts:
- J5: footprint Connector_PinHeader_2.54mm:PinHeader_2x04_P2.54mm_Vertical -> Connector_PinHeader_2.54mm:PinHeader_2x05_P2.54mm_Vertical
- Q1: footprint (none) -> Sufst_GPS:140107146000
- R3-DNC1, R4-DNC1: footprint PCM_Resistor_SMD_AKL:R_0805_2012Metric -> PCM_Resistor_SMD_AKL:R_0805_2012Metric_Pad1.15x1.40mm_HandSolder
Connections:
- net +5V renamed +5V USB
- net GPS1_RX renamed GPS1_RX_DOMI
- net GPS1_TX renamed GPS1_TX_DIMO
- net GPS2_RX renamed GPS2_TX_DIMO
- net GPS2_TX renamed GPS2_RX_DOMI
- net USB_DM renamed USB_DN
Other:
- moved on the sheet: C15
