File: sensor-pdm/linear_regulator.kicad_sch (KiCad schematic)
At the start: 0 parts

Commit message: Added sensor supply LDOs
TODO: See if LDOs are enough at dropout to handle switching noise
Parts:
- added C19: 0.1u, Capacitor_SMD:C_0603_1608Metric, symbol Device:C
- added C20: 1u, Capacitor_SMD:C_0603_1608Metric, symbol Device:C
- added JP1: SolderJumper_2_Bridged, Jumper:SolderJumper-2_P1.3mm_Bridged2Bar_RoundedPad1.0x1.5mm, symbol Jumper:SolderJumper_2_Bridged
- added R16, R17: 120k, Resistor_SMD:R_0603_1608Metric, symbol Device:R
- added U3: NCV8730, Package_DFN_QFN:DFN-6-1EP_2x2mm_P0.65mm_EP1x1.6mm, symbol SUFST:NCV8730
Connections:
- new net: JP1.1 (A), U3.4 (EN)
- new net ADJ: R16.2, R17.1, U3.2 (NC)
- new net GND: C19.1, C20.1, R17.2, U3.3 (GND), U3.7 (EX)
- new net PG: U3.5 (NC)
- new net Vin: C19.2, JP1.2 (B), U3.6 (IN)
- new net Vout: C20.2, R16.1, U3.1 (OUT)
Other:
- note added: "V_{REF} = 1.2V"

Commit message: Updated BOM, ready for review
Parts:
- C19: Mouser Part Number (none) -> 187-CL10B104KB85PNL; To Order (none) -> TRUE
- C20: Mouser Part Number (none) -> 963-UMK107BJ105KA-T; To Order (none) -> TRUE
- R16: value 120k -> 900k; Mouser Part Number (none) -> 603-RT0603FRE10100KL; To Order (none) -> INV
- R17: value 120k -> 100k; To Order (none) -> INV
- U3: Mouser Part Number (none) -> 863-NCV8730BMTWADJTB; To Order (none) -> TRUE
Changed lines of the file:
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@@
+			)
+		)
+		(property "To Order" "TRUE"
+			(at 91.44 46.99 0)
+			(effects
+				(font
+					(size 1.27 1.27)
+				)
+				(hide yes)
+			)
+		)
+		(property "Mouser Part Number" "863-NCV8730BMTWADJTB"
+			(at 91.44 46.99 0)
+			(effects
+				(font
+					(size 1.27 1.27)
+				)
+				(hide yes)
 			)
 		)
@@
 		)
 		(property "Description" "Unpolarized capacitor"
+			(at 162.56 62.23 0)
+			(effects
+				(font
+					(size 1.27 1.27)
+				)
+				(hide yes)
+			)
+		)
+		(property "To Order" "TRUE"
+			(at 162.56 62.23 0)
+			(effects
+				(font
+					(size 1.27 1.27)
+				)
+				(hide yes)
+			)
+		)
+		(property "Mouser Part Number" "963-UMK107BJ105KA-T"
 			(at 162.56 62.23 0)
 			(effects
@@
 			)
 		)
-		(property "Value" "120k"
+		(property "Value" "100k"
 			(at 144.78 69.8499 0)
 			(effects
@@
 		)
 		(property "Description" "Resistor"
+			(at 142.24 68.58 0)
+			(effects
+				(font
+					(size 1.27 1.27)
+				)
+				(hide yes)
+			)
+		)
+		(property "To Order" "INV"
 			(at 142.24 68.58 0)
 			(effects
@@
 			)
 		)
-		(property "Value" "120k"
+		(property "Value" "900k"
 			(at 144.78 57.1499 0)
 			(effects
@@
 		)
 		(property "Description" "Resistor"
+			(at 142.24 55.88 0)
+			(effects
+				(font
+					(size 1.27 1.27)
+				)
+				(hide yes)
+			)
+		)
+		(property "To Order" "INV"
+			(at 142.24 55.88 0)
+			(effects
+				(font
+					(size 1.27 1.27)
+				)
+				(hide yes)
+			)
+		)
+		(property "Mouser Part Number" "603-RT0603FRE10100KL "
 			(at 142.24 55.88 0)
 			(effects
@@
 			)
 		)
+		(property "To Order" ""
+			(at 78.105 58.42 0)
+			(effects
+				(font
+					(size 1.27 1.27)
+				)
+				(hide yes)
+			)
+		)
 		(pin "2"
 		)
@@
 			(at 55.88 57.15 0)
 			(effects
+				(font
+					(size 1.27 1.27)
+				)
+				(hide yes)
+			)
+		)
+		(property "To Order" "TRUE"
+			(at 55.88 57.15 0)
+			(effects
+				(font
+					(size 1.27 1.27)
+				)
+				(hide yes)
+			)
+		)
+		(property "Mouser Part Number" "187-CL10B104KB85PNL"
+			(at 55.88 57.15 0)
+			(effects
