File: ESF/ESF-schematics/Latching_PCB.kicad_sch (KiCad schematic)
At the start: 48 parts, among them J10 Conn_02x06, J9 Conn_02x06, K10 Relay_SPDT, K11 Relay_SPDT, Q10 XP262N7002TR-G, Q11 DMP3056L-7, Q12 XP262N7002TR-G, Q13 XP262N7002TR-G, Q14 XP262N7002TR-G, Q5 XP262N7002TR-G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

Commit message: Finished latching AMS and  IMD
Parts:
- removed K10, K11: Relay_SPDT, symbol Relay:Relay_SPDT
- added K3: AMS RLY, symbol Relay:Relay_SPST-NO
- added K5: IMD RLY, symbol Relay:Relay_SPST-NO
Connections:
- net +12V is gone; now on net +GLV: R108.2, R110.2
- net +GLV: now also K3.A1, K5.A1
- net AMS_FAULT_LATCHED: no longer Q13.1 (G), U2.13 (Q)
- net IMD_LED_K: no longer R108.1, R109.2, R110.1, R111.2
- net SHUTDOWN_IN: now also K3.14
- net SHUTDOWN_OUT: now also K5.13
- net at Q5.3 (D): now also K3.A2
- net at Q9.3 (D): now also K5.A2
- net BMS_OK_LATCHED renamed AMS_OK_LATCHED
- new net: K3.13, K5.14
- new net AMS_LED_SIGNAL: R110.1, R111.2
- new net IMD_FAULT_LATCHED: Q13.1 (G), U2.13 (Q)
- new net IMD_LED_SIGNAL: R108.1, R109.2
- no-connect marks 8 -> 6
Other:
- note added: "FSG Rule"
- note added: "FSUK RULE"
- note added: "Hence, no separate TSAL battery is used for FSG, and all circuits that use TSAL power instead powered by the LVS"
- note added: "OFF"
- note added: "ON"
- note added: "Safe State is LED on"
- note added: "active high"
