File: ESF/ESF-schematics/TSAL_RED.kicad_sch (KiCad schematic)
At the start: 59 parts, among them IC2 TPS922051D1DSGR, J3 HV+, J4 HV-, J5 Conn_01x04, Q3 IPD80R4K5P7, Q3 XP262N7002TR-G, Q4 XP262N7002TR-G, U10 40106, U13 AZ431LBNTR-G1, U14 TLP175A

Commit message: Edited text
Other:
- note added: "Flashing light operation controlled by Schmitt Trigger Oscillator. When HV_DETECTED is true, the diode is off, and the output oscillates at required 2-5 Hz frequency, with 50% duty cycle. When HV_DETECTED is false, the input to the second Schmitt inverter is pulled high, and the output is low."
- note removed: "Flashing light operation controlled by Schmitt Trigger Oscillator. When HV_DETECTED is true, the diode is off, and the output oscillates at required 2-5 Hz frequency. When HV_DETECTED is false, the input to the second Schmitt inverter is pulled high, and the output is low."
Changed lines of the file:
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@@
 		)
 	)
-	(text "Flashing light operation controlled\nby Schmitt Trigger Oscillator.\n\nWhen HV_DETECTED is true, the diode \nis off, and the output oscillates\nat required 2-5 Hz frequency.\n\nWhen HV_DETECTED is false, the input to\nthe second Schmitt inverter is pulled\nhigh, and the output is low."
+	(text "Flashing light operation controlled\nby Schmitt Trigger Oscillator.\n\nWhen HV_DETECTED is true, the diode \nis off, and the output oscillates\nat required 2-5 Hz frequency, \nwith 50% duty cycle.\n\nWhen HV_DETECTED is false, the input to\nthe second Schmitt inverter is pulled\nhigh, and the output is low."
 		(exclude_from_sim no)
-		(at 122.682 191.77 0)
+		(at 122.682 192.278 0)
 		(effects
 			(font

Commit message: Tsal stuff
Other:
- note added: "OFF"
- note added: "ON"
- note added: "Safe State is LED off"
- note added: "TSAL LED PCB - located at top of Roll Hoop"
- note added: "Weak pull down to ensure safe state if wire disconnected"
- note removed: "TSAL Driver PCB - located at top of Roll Hoop"
Changed lines of the file:
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@@
+		)
+	)
+	(text "ON"
+		(exclude_from_sim no)
+		(at 28.956 249.936 0)
+		(effects
+			(font
+				(size 2 2)
+			)
 		)
 	)
@@
 		)
 	)
-	(text "TSAL Driver PCB - located at top of Roll Hoop"
+	(text "TSAL LED PCB - located at top of Roll Hoop"
 		(exclude_from_sim no)
 		(at 79.248 206.248 0)
@@
 		)
 	)
+	(text "Weak pull down to ensure safe state\nif wire disconnected"
+		(exclude_from_sim no)
+		(at 21.59 271.78 0)
+		(effects
+			(font
+				(size 1.27 1.27)
+			)
+			(justify left)
+		)
+	)
 	(text "TS+ voltage divided across\nfive 200k Ohm resistors.\nPower dissipation divided across string\n\nEach resistor rated for 150V,\nso capable of up to 750V - above the \nmaximum 600V TS Voltage\nand can handle transients"
 		(exclude_from_sim no)
@@
 		)
 	)
+	(text "Safe State is LED off"
+		(exclude_from_sim no)
+		(at 33.02 243.84 0)
+		(effects
+			(font
+				(size 1.27 1.27)
+			)
+		)
+	)
 	(text "Flashing light operation controlled\nby Schmitt Trigger Oscillator.\n\nWhen HV_DETECTED is true, the diode \nis off, and the output oscillates\nat required 2-5 Hz frequency, \nwith 50% duty cycle.\n\nWhen HV_DETECTED is false, the input to\nthe second Schmitt inverter is pulled\nhigh, and the output is low."
 		(exclude_from_sim no)
@@
 		)
 	)
+	(text "OFF"
+		(exclude_from_sim no)
+		(at 37.338 249.936 0)
+		(effects
+			(font
+				(size 2 2)
+			)
+		)
+	)
 	(text "High Power, bright LEDs"
 		(exclude_from_sim no)
@@
 	(wire
 		(pts
-			(xy 50.165 259.08) (xy 61.595 259.08)
+			(xy 43.18 259.08) (xy 61.595 259.08)
 		)
 		(stroke
@@
 		)
 	)
+	(polyline
+		(pts
+			(xy 33.02 252.73) (xy 40.64 252.73)
+		)
+		(stroke
+			(width 0)
+			(type default)
+		)
+	)
 	(wire
 		(pts
@@
 		)
 	)
+	(polyline
+		(pts
+			(xy 33.02 246.38) (xy 33.02 252.73)
+		)
+		(stroke
+			(width 0)
+			(type default)
+		)
+	)
 	(wire
 		(pts
@@
 		(pts
 			(xy 171.45 100.33) (xy 171.45 101.6)
+		)
+		(stroke
+			(width 0)
+			(type default)
+		)
+	)
+	(polyline
+		(pts
+			(xy 25.4 246.38) (xy 33.02 246.38)
 		)
 		(stroke
@@
 	)
 	(label "RED_LED_ENABLED"
-		(at 50.165 259.08 180)
-		(effects
-			(font
+		(at 43.18 259.08 180)
+		(effects
+			(font

Commit message: finish tsal green
Parts:
- removed C17: 100n, Capacitor_SMD:C_0805_2012Metric_Pad1.18x1.45mm_HandSolder, symbol Device:C
- removed C18: 10u, Capacitor_SMD:C_0805_2012Metric_Pad1.18x1.45mm_HandSolder, symbol Device:C
- removed C19, C20, C21: 10u, Capacitor_SMD:C_0603_1608Metric, symbol Device:C
- removed C20, C22, C27: 22u, Capacitor_SMD:C_0805_2012Metric, symbol Device:C
- removed C22, C23, C26: 0.1u, Capacitor_SMD:C_0603_1608Metric, symbol Device:C
- removed C24, C25: 1n, Capacitor_SMD:C_0603_1608Metric, symbol Device:C
- removed D12, D13: 1.5SMC300CA, PCM_Diode_SMD_AKL:D_SMC_TVS, symbol PCM_Diode_TVS_AKL:1.5SMC300CA
- removed D14: MMSZ4699T1G, Diode_SMD:D_SOD-123, symbol Diode:1N630xA
- removed D15: MMSZ4684-E3-08, Diode_SMD:D_SOD-123, symbol Diode:1N630xA
- removed D16: BAT54W, Package_TO_SOT_SMD:SOT-323_SC-70, symbol Diode:BAT54W
- removed D17: SS34, Diode_SMD:D_SMA, symbol Diode:SS34
- removed D18, D19, D20, D21: SST-20-DR-A120, SUFST:Luminus_SST10_20_3030_pad, symbol Device:LED_Pad
- removed F4: 0461.500ER, SUFST:Littelfuse-04611-25ER, symbol Device:Fuse
- removed F5: 150ma, Fuse:Fuse_0805_2012Metric, symbol Device:Fuse_Small
- removed IC2: TPS922051D1DSGR, Package_SON:Texas_DSG0008A_WSON-8-1EP_2x2mm_P0.5mm_EP0.9x1.6mm, symbol sufst:TPS922051D2DSGR
- removed J3: HV+, SUFST:Molex_Micro-Fit_3.0_43045-0212_2x01_P3.00mm_Vertical, symbol Connector_Generic:Conn_01x02
- removed J4: HV-, SUFST:Molex_Micro-Fit_3.0_43045-0212_2x01_P3.00mm_Vertical, symbol Connector_Generic:Conn_01x02
- removed J5: Conn_01x04, SUFST:Molex_Micro-Fit_3.0_43045-0412_2x02_P3.00mm_Vertical, symbol Connector_Generic:Conn_01x04
- removed L2: 22u, Inductor_SMD:L_Coilcraft_XAL5030-XXX, symbol Device:L
- removed Q3, Q4: XP262N7002TR-G, Package_TO_SOT_SMD:SOT-23, symbol Device:Q_NMOS_GSD
- removed Q3: IPD80R4K5P7, Package_TO_SOT_SMD:TO-252-2, symbol SUFST:FQD1N80TM
- removed R1: 1k, Resistor_SMD:R_2512_6332Metric, symbol Device:R
- removed R55, R56, R57, R58, R59, R61: 200k, Resistor_SMD:R_0805_2012Metric_Pad1.20x1.40mm_HandSolder, symbol Device:R
- removed R60: 33k, Resistor_SMD:R_0805_2012Metric_Pad1.20x1.40mm_HandSolder, symbol Device:R
- removed R62, R65, R67, R68: 10k, Resistor_SMD:R_0805_2012Metric_Pad1.20x1.40mm_HandSolder, symbol Device:R
- removed R63: 47k, Resistor_SMD:R_0805_2012Metric_Pad1.20x1.40mm_HandSolder, symbol Device:R
- removed R64, R66: 1k, Resistor_SMD:R_0805_2012Metric_Pad1.20x1.40mm_HandSolder, symbol Device:R
- removed R69: 150k, Resistor_SMD:R_0805_2012Metric_Pad1.20x1.40mm_HandSolder, symbol Device:R
- removed R70: 470, Resistor_SMD:R_0805_2012Metric_Pad1.20x1.40mm_HandSolder, symbol Device:R
- removed R71: 100k, Resistor_SMD:R_0603_1608Metric, symbol Device:R
- removed R72, R73, R75: 100, Resistor_SMD:R_0603_1608Metric, symbol Device:R
- removed R74: 200m, Resistor_SMD:R_1206_3216Metric, symbol Device:R
- removed RV5: 470k, Potentiometer_THT:Potentiometer_Bourns_3296W_Vertical, symbol Device:R_Potentiometer
- removed U10: 40106, Package_SO:SOIC-14_3.9x8.7mm_P1.27mm, symbol 4xxx:40106
- removed U13: AZ431LBNTR-G1, Package_TO_SOT_SMD:SOT-23_Handsoldering, symbol SUFST:AZ431LBNTR-G1
- removed U14: TLP175A, Package_SO:MFSOP6-4_4.4x3.6mm_P1.27mm, symbol Relay_SolidState:TLP175A
- added C100, C89, C90, C91: 100n, Capacitor_SMD:C_0805_2012Metric_Pad1.18x1.45mm_HandSolder, symbol Device:C
- added C101, C102, C75, C76: 1n, Capacitor_SMD:C_0603_1608Metric, symbol Device:C
- added C103, C73, C74, C77, C98, C99: 0.1u, Capacitor_SMD:C_0603_1608Metric, symbol Device:C
- added C104, C105, C106, C78, C79, C80: 22u, Capacitor_SMD:C_0805_2012Metric, symbol Device:C
- added C107, C83, C84, C85, C86, C94: 10u, Capacitor_SMD:C_0805_2012Metric_Pad1.18x1.45mm_HandSolder, symbol Device:C
- added C62, C68, C69, C95, C96, C97: 10u, Capacitor_SMD:C_0603_1608Metric, symbol Device:C
- added C81: 10u, Capacitor_SMD:C_0805_2012Metric_Pad1.18x1.45mm_HandSolder, symbol Device:C_Small
- added C82, C87: 100n, Capacitor_SMD:C_0805_2012Metric_Pad1.18x1.45mm_HandSolder, symbol Device:C_Small
- added C88: 1u, Capacitor_SMD:C_0805_2012Metric_Pad1.18x1.45mm_HandSolder, symbol Device:C_Small
- added C92, C93: 100u, Capacitor_THT:CP_Radial_D5.0mm_P2.00mm, symbol Device:C_Polarized
- added D100, D101, D98, D99: SST-20-DR-A120, SUFST:Luminus_SST10_20_3030_pad, symbol Device:LED_Pad
- added D54, D96: SS34, Diode_SMD:D_SMA, symbol Diode:SS34
- added D55, D56, D57, D66: SST-10-G-A120, SUFST:Luminus_SST10_20_3030_pad, symbol Device:LED_Pad
- added D67, D68, D69, D70, D71, D74, D88: D_TVS, symbol Device:D_TVS
- added D72, D73, D92, D93: 1.5SMC300CA, PCM_Diode_SMD_AKL:D_SMC_TVS, symbol PCM_Diode_TVS_AKL:1.5SMC300CA
- added D75, D78, D79, D80, D81, D82, D83, D84, D97: BAT54W, Package_TO_SOT_SMD:SOT-323_SC-70, symbol Diode:BAT54W
- added D76, D94: MMSZ4699T1G, Diode_SMD:D_SOD-123, symbol Diode:1N630xA
- added D77, D95: MMSZ4684-E3-08, Diode_SMD:D_SOD-123, symbol Diode:1N630xA
- added D85: GREEN, LED_SMD:LED_0603_1608Metric, symbol Device:LED
- added D86: SS14+, Diode_SMD:D_SMA, symbol Device:D
- added D87: RED, LED_SMD:LED_0603_1608Metric, symbol Device:LED
- added D89: BLUE, LED_SMD:LED_0603_1608Metric, symbol Device:LED
- added D90: YELLOW, LED_SMD:LED_0603_1608Metric, symbol Device:LED
- added D91: ORANGE, LED_SMD:LED_0603_1608Metric, symbol Device:LED
- added F11, F17: 0461.500ER, SUFST:Littelfuse-04611-25ER, symbol Device:Fuse
- added F14, F15: 0448.500MR, Fuse:Fuse_Littelfuse-NANO2-451_453, symbol Device:Fuse
- added F16, F18: 150ma, Fuse:Fuse_0805_2012Metric, symbol Device:Fuse_Small
- added GRN2, IMP2: TestPoint, TestPoint:TestPoint_Pad_D1.5mm, symbol Connector:TestPoint
- added IC3, IC4: TPS922051D1DSGR, Package_SON:Texas_DSG0008A_WSON-8-1EP_2x2mm_P0.5mm_EP0.9x1.6mm, symbol sufst:TPS922051D2DSGR
- added J17, J25: HV+, SUFST:Molex_Micro-Fit_3.0_43045-0212_2x01_P3.00mm_Vertical, symbol Connector_Generic:Conn_01x02
- added J18, J26: HV-, SUFST:Molex_Micro-Fit_3.0_43045-0212_2x01_P3.00mm_Vertical, symbol Connector_Generic:Conn_01x02
- added J19: Conn_01x02, symbol Connector_Generic:Conn_01x02
- added J20, J22: Conn_01x03, symbol Connector_Generic:Conn_01x03
- added J21, J23: Conn_01x01, symbol Connector_Generic:Conn_01x01
- added J24, J27: Conn_01x04, SUFST:Molex_Micro-Fit_3.0_43045-0412_2x02_P3.00mm_Vertical, symbol Connector_Generic:Conn_01x04
- added L3, L4: 22u, Inductor_SMD:L_Coilcraft_XAL5030-XXX, symbol Device:L
- added NT1, NT2, NT3, NT4: NetTie_2, NetTie:NetTie-2_SMD_Pad0.5mm, symbol Device:NetTie_2
- added Q20, Q23: IPD80R4K5P7, Package_TO_SOT_SMD:TO-252-2, symbol SUFST:FQD1N80TM
- added Q21, Q22, Q24, Q25: XP262N7002TR-G, Package_TO_SOT_SMD:SOT-23, symbol Device:Q_NMOS_GSD
- added R132, R133, R135, R204, R206, R208: 100, Resistor_SMD:R_0603_1608Metric, symbol Device:R
- added R132, R193: 100k, Resistor_SMD:R_0603_1608Metric, symbol Device:R
- added R134, R207: 200m, Resistor_SMD:R_1206_3216Metric, symbol Device:R
- added R153, R215: 5.6k, Resistor_SMD:R_0805_2012Metric_Pad1.20x1.40mm_HandSolder, symbol Device:R
- added R154, R216: 3.9k, Resistor_SMD:R_0805_2012Metric_Pad1.20x1.40mm_HandSolder, symbol Device:R
- added R155, R194: 1k, Resistor_SMD:R_2512_6332Metric, symbol Device:R
- added R156: 1k, Resistor_SMD:R_0805_2012Metric_Pad1.20x1.40mm_HandSolder, symbol Device:R_Small
- added R157: 47k, Resistor_SMD:R_0805_2012Metric_Pad1.20x1.40mm_HandSolder, symbol Device:R_Small
- added R158, R159, R166, R167, R178: 10k, Resistor_SMD:R_0805_2012Metric_Pad1.20x1.40mm_HandSolder, symbol Device:R_Small
- added R160, R161, R162, R163, R164, R168, R197, R198, R199, R200, R201, R203: 200k, Resistor_SMD:R_0805_2012Metric_Pad1.20x1.40mm_HandSolder, symbol Device:R
- added R165, R202: 33k, Resistor_SMD:R_0805_2012Metric_Pad1.20x1.40mm_HandSolder, symbol Device:R
- added R169: 100k, Resistor_SMD:R_0805_2012Metric_Pad1.20x1.40mm_HandSolder, symbol Device:R
- added R170, R171, R172, R174, R177, R179, R180, R181, R182, R186, R189, R195, R196, R205, R213: 10k, Resistor_SMD:R_0805_2012Metric_Pad1.20x1.40mm_HandSolder, symbol Device:R
- added R173, R176: 270, Resistor_SMD:R_2512_6332Metric, symbol Device:R
- added R175: 100k, Resistor_SMD:R_0805_2012Metric_Pad1.20x1.40mm_HandSolder, symbol Device:R_Small
- added R183, R187, R190, R191, R192: 10k, Resistor_SMD:R_0603_1608Metric_Pad0.98x0.95mm_HandSolder, symbol Device:R
- added R184, R209: 47k, Resistor_SMD:R_0805_2012Metric_Pad1.20x1.40mm_HandSolder, symbol Device:R
- added R185, R188, R211, R214: 1k, Resistor_SMD:R_0805_2012Metric_Pad1.20x1.40mm_HandSolder, symbol Device:R
- added R210: 150k, Resistor_SMD:R_0805_2012Metric_Pad1.20x1.40mm_HandSolder, symbol Device:R
- added R212: 470, Resistor_SMD:R_0805_2012Metric_Pad1.20x1.40mm_HandSolder, symbol Device:R
- added RV6: 470k, Potentiometer_THT:Potentiometer_Bourns_3296W_Vertical, symbol Device:R_Potentiometer
- added TP1: +AIR_INTENDED, TestPoint:TestPoint_Pad_D1.5mm, symbol Connector:TestPoint
- added TP2: -AIR_INTENDED, TestPoint:TestPoint_Pad_D1.5mm, symbol Connector:TestPoint
- added TP3: PRCHG_INTENDED, TestPoint:TestPoint_Pad_D1.5mm, symbol Connector:TestPoint
- added U21, U23, U30, U31, U33: 40106, Package_SO:SOIC-14_3.9x8.7mm_P1.27mm, symbol 4xxx:40106
- added U24: 4071, Package_SO:SOIC-14_3.9x8.7mm_P1.27mm, symbol 4xxx:4071
- added U25, U29, U37: 4081, Package_SO:SOIC-14_3.9x8.7mm_P1.27mm, symbol 4xxx:4081
- added U32, U38: AZ431LBNTR-G1, Package_TO_SOT_SMD:SOT-23_Handsoldering, symbol SUFST:AZ431LBNTR-G1
- added U34, U39: TLP175A, Package_SO:MFSOP6-4_4.4x3.6mm_P1.27mm, symbol Relay_SolidState:TLP175A
- added U35, U36: 4013, Package_SO:SOIC-14_3.9x8.7mm_P1.27mm, symbol 4xxx:4013
Connections:
- net +GLV: now also C103.1, C104.1, C105.1, C106.1, C62.1, C68.2, C69.1, C73.2, C77.1, C78.1, C79.1, C80.1, C95.1, C96.2, C97.1, C98.2, D54.1 (K), D55.2 (A), D56.2 (A), D96.1 (K), D98.2 (A), D99.2 (A), F15.1, F16.2, F18.2, IC3.2 (VIN), IC4.2 (VIN), R135.2, R185.1, R188.1, R208.2, R211.1, R214.1, U34.6, U39.6
- net GND: now also C100.2, C101.2, C107.2, C62.2, C68.1, C69.2, C73.1, C74.2, C75.2, C81.2, C82.1, C83.2, C84.2, C85.2, C86.2, C87.1, C88.2, C89.2, C90.2, C91.2, C92.2, C93.2, C94.2, C95.2, C96.1, C97.2, C98.1, C99.2, D100.3 (PAD), D101.3 (PAD), D55.3 (PAD), D56.3 (PAD), D57.3 (PAD), D66.3 (PAD), D67.2 (A2), D68.2 (A2), D69.1 (A1), D70.1 (A1), D71.2 (A2), D74.1 (A1), D88.1 (A1), D98.3 (PAD), D99.3 (PAD), IC3.1 (GND), IC3.9 (EP), IC4.1 (GND), IC4.9 (EP), J24.4 (Pin_4), J27.4 (Pin_4), Q21.2 (S), Q22.2 (S), Q24.2 (S), Q25.2 (S), R132.1, R154.1, R156.2, R158.2, R159.2, R178.2, R183.2, R184.1, R186.1, R187.2, R190.2, R191.2, R192.2, R193.1, R195.1, R209.1, R213.1, R216.1, U35.6 (S), U36.3 (C), U36.5 (D)
- net HV+: now also F11.2, F17.2, J17.1 (Pin_1), J25.1 (Pin_1)
- net HV-: now also D73.1 (K), D77.2 (A2), D93.1 (K), D95.2 (A2), J18.2 (Pin_2), J26.2 (Pin_2), R165.2, R168.2, R202.2, R203.2, U32.3 (A), U38.3 (A)
- net HV_DETECTED: now also J24.1 (Pin_1), J27.1 (Pin_1), Q22.3 (D), Q25.3 (D), R188.2, R195.2, R196.2, R214.2
- net HV_FUSED: now also D72.2 (A), D92.2 (A), Q20.2 (D), Q23.2 (D), R155.1, R160.2, R194.1, R197.2
- net RED_LED_ENABLED: now also R210.2, R215.2, RV6.1, U23.4
- net ~{HV_DETECTED}: now also D68.1 (A1), J21.1 (Pin_1), J24.2 (Pin_2), J27.2 (Pin_2), Q21.3 (D), Q22.1 (G), Q24.3 (D), Q25.1 (G), R185.2, R186.2, R211.2, R213.2, U25.13, U29.2
- new net: F11.1, R155.2
- new net: R197.1, R198.1
- new net: R198.2, R199.2
- new net: D87.1 (K), R187.1
- new net: D91.1 (K), R192.1
- new net: D86.1 (K), F14.1
- new net: D96.2 (A), IC4.8 (SW), L4.1
- new net: L4.2, R206.2, R207.1
- new net: D94.2 (A2), D95.1 (A1), R202.1, U38.1 (REF)
- new net: C102.2, C103.2, C104.2, C105.2, C106.2, D100.1 (K), D101.1 (K), IC4.6 (CSP), R207.2, R208.1
- new net: D100.2 (A), D101.2 (A), D98.1 (K), D99.1 (K)
- new net: Q23.3 (S), R203.1, R205.1
- new net: R205.2, U39.1
- new net: D97.3 (K), R210.1, R212.2, RV6.2, RV6.3, U23.3
- new net: D94.1 (A1), Q23.1 (G), R201.1
- new net: Q24.1 (G), R209.2, U39.4
- new net: U38.2 (K), U39.3
- new net: Q20.3 (S), R168.1, R174.1
- new net: C75.1, R132.1
- new net: IC3.5 (COMP), R132.2
- new net: C82.2, R167.2
- new net: C102.1, IC4.7 (CSN), R206.1
- new net: U23.11, U23.12
- new net: D92.1 (K), D93.2 (A)
- new net: F16.1, J24.3 (Pin_3)
- new net: R174.2, U34.1
- new net: C107.1, R212.1
- new net: R199.1, R200.1
- new net: R200.2, R201.2
- new net: Q21.1 (G), R184.2, U34.4
- new net: D76.1 (A1), Q20.1 (G), R164.1
- new net: C87.2, R166.2
- new net: C99.1, IC4.4 (VCC)
- new net: D76.2 (A2), D77.1 (A1), R165.1, U32.1 (REF)
- new net: C76.2, C77.2, C78.2, C79.2, C80.2, D57.1 (K), D66.1 (K), IC3.6 (CSP), R134.2, R135.1
- new net: D55.1 (K), D56.1 (K), D57.2 (A), D66.2 (A)
- new net: D90.1 (K), R191.1
- new net: IC4.5 (COMP), R204.2
- new net: D54.2 (A), IC3.8 (SW), L3.1
- new net: U32.2 (K), U34.3
- new net: D85.1 (K), R183.1
- new net: C100.1, R196.1, U23.1
- new net: D97.1 (A), U23.2
- new net: R162.1, R163.1
- new net: R163.2, R164.2
- new net: L3.2, R133.2, R134.1
- new net: D89.1 (K), R190.1
- new net: F18.1, J27.3 (Pin_3)
- new net: R161.2, R162.2
- new net: D72.1 (K), D73.2 (A)
- new net: C101.1, R204.1
- new net: C74.1, IC3.4 (VCC)
- new net: C76.1, IC3.7 (CSN), R133.1
- new net: F17.1, R194.2
- new net: R160.1, R161.1
- new net +12V: C92.1, D88.2 (A2), F14.2, R173.1, R176.1, R177.1, U35.5 (D)
- new net +AIR_MECH_IMP: R172.1, U29.11
- new net +AIR_MECH_IMP_RC: C85.1, R172.2, U33.5
- new net +GLV_FUSED: C93.1, F15.2, R179.2, R189.2
- new net -AIR_MECH_IMP: R171.1, U29.10
- new net -AIR_MECH_IMP_RC: C84.1, R171.2, U33.3
- new net AIRS_CLSD: U25.3, U29.1
- new net CLOSE_NEG_AIR: NT1.2, NT3.2
- new net CLOSE_PCHG_RLY: NT4.2, U37.11
- new net CLOSE_POS_AIR: NT2.2, U37.10
- new net GREEN_LED_ENABLED: R153.2, U23.10
- new net GREEN_LED_ENABLED_5V: IC3.3 (DIM), R132.2, R153.1, R154.2
- new net GREEN_LED_ON: D70.2 (A2), D85.2 (A), GRN2.1, J20.3 (Pin_3), U23.13, U31.12
- new net HIGH_AIR_INTENDED_ON: D89.2 (A), NT2.1, TP1.1, U24.1, U29.12
- new net HS_ACTIVE: U24.3, U25.1
- new net HV_IMP: R169.1, U29.3
- new net HV_IMP_RC: C86.1, R169.2, U33.9
- new net IMPLAUSIBLE: D87.2 (A), IMP2.1, U24.6, U36.1 (Q)
- new net IMP_TRIG: U33.10, U36.6 (S)
- new net INV_CLOSE_MAIN_CONTACTOR: D71.1 (A1), J19.2 (Pin_2), R158.1, R167.1, U37.9
- new net INV_CLOSE_PCHG_RLY: D74.2 (A2), J19.1 (Pin_1), R159.1, R166.1, U37.13
- new net LOW_AIR_INTENDED_ON: D90.2 (A), NT3.1, TP2.1, U25.2, U29.8
- new net POR: D80.1 (A), U21.10, U30.10, U30.5, U36.4 (R)
- new net POR_RC: C81.1, D75.1 (A), R157.1, U30.11
- new net PRCHG_INTENDED_ON: D91.2 (A), NT4.1, TP3.1, U24.2, U29.6
- new net PRCHG_MECH_IMP: R170.1, U29.4
- new net PRCHG_MECH_IMP_RC: C83.1, R170.2, U33.1
- new net RED_LED_ENABLED_5V: IC4.3 (DIM), R193.2, R215.1, R216.2
- new net SHUTDOWN: D75.3 (K), D86.2 (A), J23.1 (Pin_1), R156.1, R157.2
- new net TSAL_POR_RC: C94.1, R189.1, U21.11
- new net TS_ENABLED: NT1.1, U35.1 (Q), U37.12, U37.8
- new net TS_EN_POR: D79.3 (K), D80.3 (K), R178.1, U35.4 (R)
- new net TS_EN_RISING: U30.8, U35.3 (C)
- new net TS_OFF: U25.10, U31.1
- new net TS_ON_INPUT: D69.2 (A2), J20.2 (Pin_2), U30.13
- new net TS_ON_RC: C88.1, D78.3 (K), R175.1, U30.9
- new net TS_READY: D67.1 (A1), J20.1 (Pin_1), U30.6
- new net TS_UNSAFE: U24.5, U31.2
- new net ~{+AIR_MECH_HV}: U25.11, U25.9
- new net ~{+AIR_MECH_IMP}: D83.3 (K), U33.6
- new net ~{-AIR_MECH_IMP}: D82.3 (K), U33.4
- new net ~{-AIR_PRCHG_MECH}: U25.4, U25.8
- new net ~{-PRCHG_MECH_IMP}: D81.3 (K), U33.2
- new net ~{HIGH_AIR_MECH_ON_IN}: J22.2 (Pin_2), R176.2, R181.2
- new net ~{HIGH_AIR_MECH_ON}: C90.1, R181.1, U25.12, U29.13
- new net ~{HV_IMP}: D84.3 (K), U33.8
- new net ~{IMP_TRIG}: D81.1 (A), D82.1 (A), D83.1 (A), D84.1 (A), R179.1, U33.11
- new net ~{LOW_AIR_MECH_ON_IN}: J22.1 (Pin_1), R173.2, R180.2
- new net ~{LOW_AIR_MECH_ON}: C91.1, R180.1, U25.6, U29.9
- new net ~{PRCHG_MECH_ON_IN}: J22.3 (Pin_3), R177.2, R182.2
- new net ~{PRCHG_MECH_ON}: C89.1, R182.1, U25.5, U29.5
- new net ~{TSAL_IMP}: U24.4, U31.13
- new net ~{TS_ON}: D78.1 (A), D79.1 (A), R175.2, U30.12
- no-connect marks 2 -> 6
Other:
- note added: "...and this point to go high"
- note added: "0.5A"
- note added: "Any implausibility causes this point to go low"
- note added: "Auxillary contacts (AIRs and precharge)"
- note added: "Close the +ve AIR when the TS is enabled and the inverter commands main contactor closed"
- note added: "Close the -ve AIR when the TS is enabled"
- note added: "Close the pre-charge relay when the TS is enabled and the inverter commands it closed"
- note added: "Diode prevents capacitors from powering the shutdown loop when the shutdown loop opens, without it the capacitors on the 12V supply of this board would keep the AIRs on for a short time after the loop opens"
- note added: "ERR"
- note added: "For this to go high, the following must be true: - TS_ON is high (else the latch will be in reset). - The shutdown loop has been closed for at least 0.47s (else the latch will be in reset). - A rising edge on TS_ON has been detected at least 0.47s after the shutdown circuit was last open. This last point guarantees rule EV4.11.4 (FSUK 2024)"
- note added: "From Motor Controller"
- note added: "GREEN_LED_ON - true unless TSAC_ACTIVE or IMPLAUSIBLE."
- note added: "Goes high 0.1s after TS_ON goes high. Goes low immediately after TS_ON goes low. Rising edge here turns latch on, unless it's held in reset. Delay required to ensure rising edge happens after reset goes low."
- note added: "Goes low 0.47s after shutdown circuit closes. Goes high 0.01s after shutdown circuit opens."
- note added: "HV Detection PCB - located within Accumulator, measuring vehicle side of AIRs"
- note added: "High Voltage Not Detected Signal"
- note added: "High when TS_ON is low. Also high for 0.47s after the shutdown circuit closes. Holds latch in reset while high."
- note added: "If one of the high relays is on, and the low relay is on, but no high voltage is detected for more than ~1s, that implies an implausibility."
- note added: "Low when TS_ON is high. High when TS_ON is low."
- note added: "OK"
- note added: "Power On Reset"
- note added: "Pullups to provide auxiliary contacts a "wetting current" to prevent issues with contact oxidation in the long term"
- note added: "RC=0.1s"
- note added: "RC=0.47s"
- note added: "Rules: - The TS should never be enabled if TS_ON is low - The TS should only be enabled after a rising edge of the TS_ON input. Whenever the shutdown circuit is opened, the TS should remain off until a rising edge is detected."
- note added: "SCS: - Green LED turns on when HV not detected. Safe state = off, so Green LED uses ~{HV_DETECTED} signal (short to GND means off = safe state)"
- note added: "Safe state is LED off"
- note added: "Signal from VCU when driver initiates TSON"
- note added: "Signal to VCU when TS able to start"
- note added: "TS OFF"
- note added: "TS ON"
- note added: "TSAL GREEN Signal to TSAL Logic PCB"
- note added: "Time constant 1ms rise, 2ms fall (through pull-down resistor). Asymmetry not ideal, but not a problem because the signals are slow."
- note added: "To ensure signal voltage"
- note added: "Tractive Relay Controller PCB - AIR Control Logic"
- note added: "Tractive Relay Controller PCB - GREEN Light Implausibility Check"
- note added: "Tractive Relay Controller PCB - Inputs and Outputs"
- note added: "Voltage Divider to 5V for LED driver pin"
