File: ESF/ESF-schematics/TSAL_GREEN_ACCU.kicad_sch (KiCad schematic)
At the start: 113 parts, among them J17 HV+, J18 HV-, J19 Conn_01x02, J20 Conn_01x03, J21 Conn_01x01, J22 Conn_01x03, J23 Conn_01x01, J24 Conn_01x04, Q20 IPD80R4K5P7, Q21 XP262N7002TR-G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

Commit message: finish tsal
Other:
- note added: "For this to go high, the following must be true: - TS_ON is high (else the latch will be in reset). - The shutdown loop has been closed for at least 0.47s (else the latch will be in reset). - A rising edge on TS_ON has been detected at least 0.47s after the shutdown circuit was last open. This last point guarantees rule EV4.11.4 (FSG 2026)"
- note removed: "For this to go high, the following must be true: - TS_ON is high (else the latch will be in reset). - The shutdown loop has been closed for at least 0.47s (else the latch will be in reset). - A rising edge on TS_ON has been detected at least 0.47s after the shutdown circuit was last open. This last point guarantees rule EV4.11.4 (FSUK 2024)"
Changed lines of the file:
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@@
 		)
 	)
-	(text "For this to go high, the\nfollowing must be true:\n- TS_ON is high (else the\n  latch will be in reset).\n- The shutdown loop has\n  been closed for at least\n  0.47s (else the latch will\n  be in reset).\n- A rising edge on TS_ON\n  has been detected at least\n  0.47s after the shutdown\n  circuit was last open.\n\nThis last point guarantees\nrule EV4.11.4 (FSUK 2024)\n"
+	(text "For this to go high, the\nfollowing must be true:\n- TS_ON is high (else the\n  latch will be in reset).\n- The shutdown loop has\n  been closed for at least\n  0.47s (else the latch will\n  be in reset).\n- A rising edge on TS_ON\n  has been detected at least\n  0.47s after the shutdown\n  circuit was last open.\n\nThis last point guarantees\nrule EV4.11.4 (FSG 2026)\n"
 		(exclude_from_sim no)
 		(at 200.66 337.82 0)

Commit message: tsal final final final no take backs
Parts:
- added R1: 10k, Resistor_SMD:R_0805_2012Metric_Pad1.20x1.40mm_HandSolder, symbol Device:R_Small
Connections:
- net GND: now also R1.2
- net ~{HV_DETECTED}: now also R1.1
Other:
- note added: "12V Zener clamps gate voltage of Q20 to 12V, and prevents noise or low voltage accidentally triggering "HV Detected" signal until 12V gate voltage. Starts conducting at 12V. Once voltage through D76 creates 1.24V drop across R165, U32 turns on like a low side switch."
- note added: "3.3V Zener Diode D77 protect inputs to U13, clamping voltage to 3.3V"
- note added: "Pull down to ensure SCS Wire disconnect = short to GND GREEN LED off - Safe state"
- note removed: "12V Zener clamps gate voltage of Q3 to 12V, and prevents noise or low voltage accidentally triggering "HV Detected" signal until 12V gate voltage. Starts conducting at 12V. Once voltage through D14 creates 1.24V drop across R60, U13 turns on like a low side switch."
- note removed: "3.3V Zener Diode D15 protect inputs to U13, clamping voltage to 3.3V"
