File: gps-mainboard/gps-mainboard.kicad_sch (KiCad schematic)
At the start: 76 parts, among them J1 21992304, J2 Conn_01x08_Socket, Q1 2N7002, Q2 DMP510DL-7, SW1 KMR2, SW2 KMR2, U1 STM32G431C8Tx, U10 TLV75533PDYD, U13 TVS1800DRV, U21 MCP9800Ax-xOT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

Commit message: Rename project
Other:
- note added: "Debug"
- note added: "IMU and Magnetometer"
- note added: "Inputs and Outputs"
- note added: "LEDs & Button"
- note added: "Micromod Connector"
- note added: "Mounting Holes"
- note added: "STM32 MCU"
- note added: "Temperature Sensor"
- note added: "UART Direction Selection"
Changed lines of the file:
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@@
 		(comment 1 "STAG 12")
 		(comment 2 "Adam Eastman")
+		(comment 3 "Annabel Owen, Ray Wang")
 	)
 	(rectangle
@@
 		)
 	)
+	(text "Temperature Sensor"
+		(exclude_from_sim no)
+		(at 19.558 253.238 0)
+		(effects
+			(font
+				(size 1.778 1.778)
+			)
+			(justify left bottom)
+		)
+	)
 	(text "Route through unused pins"
 		(exclude_from_sim no)
@@
 		)
 	)
+	(text "LEDs & Button"
+		(exclude_from_sim no)
+		(at 129.286 221.234 0)
+		(effects
+			(font
+				(size 1.778 1.778)
+			)
+			(justify left bottom)
+		)
+	)
+	(text "Debug"
+		(exclude_from_sim no)
+		(at 19.812 220.98 0)
+		(effects
+			(font
+				(size 1.778 1.778)
+			)
+			(justify left bottom)
+		)
+	)
 	(text "Pull up resistors\nprovided on GPS board"
 		(exclude_from_sim no)
@@
 		)
 	)
+	(text "IMU and Magnetometer"
+		(exclude_from_sim no)
+		(at 183.388 159.258 0)
+		(effects
+			(font
+				(size 1.778 1.778)
+			)
+			(justify left bottom)
+		)
+	)
 	(text "Nreset when pin \npulled low"
 		(exclude_from_sim no)
@@
 		)
 	)
+	(text "Mounting Holes"
+		(exclude_from_sim no)
+		(at 279.654 221.488 0)
+		(effects
+			(font
+				(size 1.778 1.778)
+			)
+			(justify left bottom)
+		)
+	)
 	(text "Normally pulled up to 5V on GPS board\nSetting pin 9 high turns off GPS board\nwith exception to EEPROM or RTC battery"
 		(exclude_from_sim no)
@@
 		)
 	)
+	(text "Inputs and Outputs"
+		(exclude_from_sim no)
+		(at 279.908 159.004 0)
+		(effects
+			(font
+				(size 1.778 1.778)
+			)
+			(justify left bottom)
+		)
+	)
 	(text "5V - 3.3V LDO"
 		(exclude_from_sim no)
@@
 		)
 	)
+	(text "Micromod Connector"
+		(exclude_from_sim no)
+		(at 280.416 22.86 0)
+		(effects
+			(font
+				(size 1.778 1.778)
+			)
+			(justify left bottom)
+		)
+	)
 	(text "GLV - 5V Buck Converter"
 		(exclude_from_sim no)
@@
 		)
 	)
+	(text "UART Direction Selection"
+		(exclude_from_sim no)
+		(at 19.558 159.512 0)
+		(effects
+			(font
+				(size 1.778 1.778)
+			)
+			(justify left bottom)
+		)
+	)
+	(text "STM32 MCU"
+		(exclude_from_sim no)
+		(at 109.474 21.59 0)
+		(effects
+			(font
+				(size 1.778 1.778)
+			)
+			(justify left bottom)
+		)
+	)
 	(text "GPS I2C Address 0x42"
 		(exclude_from_sim no)
@@
 		)
 		(instances
-			(project "micromod-gps"
+			(project "gps-mainboard"
 				(path "/de1c89a8-60ad-4219-8e58-e4b5538835d9"
 					(page "3")
@@
 		)
 		(instances
-			(project "micromod-gps"
+			(project "gps-mainboard"
 				(path "/de1c89a8-60ad-4219-8e58-e4b5538835d9"
 					(page "2")

Commit message: Fix ERC errors
Changed lines of the file:
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@@
 	)
 	(junction
-		(at 73.66 126.365)
-		(diameter 0)
-		(color 0 0 0 0)
-	)
-	(junction
 		(at 56.515 36.83)
 		(diameter 0)
@@
 		(color 0 0 0 0)
 	)
+	(junction
+		(at 23.495 30.48)
+		(diameter 0)
+		(color 0 0 0 0)
+	)
 	(no_connect
 		(at 343.535 47.625)
@@
 	(wire
 		(pts
+			(xy 23.495 29.21) (xy 23.495 30.48)
+		)
+		(stroke
+			(width 0)
+			(type default)
+		)
+	)
+	(wire
+		(pts
 			(xy 85.09 106.045) (xy 90.17 106.045)
 		)
@@
 	(wire
 		(pts
-			(xy 73.66 126.365) (xy 70.485 126.365)
+			(xy 70.485 126.365) (xy 83.185 126.365)
 		)
 		(stroke
@@
 	(wire
 		(pts
+			(xy 23.495 30.48) (xy 23.495 36.83)
+		)
+		(stroke
+			(width 0)
+			(type default)
+		)
+	)
+	(wire
+		(pts
 			(xy 154.305 29.21) (xy 164.465 29.21)
 		)
@@
 	(wire
 		(pts
+			(xy 23.495 36.83) (xy 24.13 36.83)
+		)
+		(stroke
+			(width 0)
+			(type default)
+		)
+	)
+	(wire
+		(pts
 			(xy 39.37 126.365) (xy 48.26 126.365)
 		)
@@
 	(wire
 		(pts
-			(xy 83.185 126.365) (xy 73.66 126.365)
-		)
-		(stroke
-			(width 0)
-			(type default)
-		)
-	)
-	(wire
-		(pts
 			(xy 293.37 131.445) (xy 293.37 133.985)
 		)
@@
 	(wire
 		(pts
-			(xy 22.86 36.83) (xy 24.13 36.83)
-		)
-		(stroke
-			(width 0)
-			(type default)
-		)
-	)
-	(wire
-		(pts
 			(xy 225.425 81.28) (xy 207.645 81.28)
 		)
@@
 		(on_board yes)
 		(dnp no)
-		(fields_autoplaced yes)
 		(property "Reference" "F1"
-			(at 27.94 31.115 90)
+			(at 27.94 33.02 90)
 			(effects
 				(font
@@
 		)
 		(property "Value" "Fuse"
-			(at 27.94 33.655 90)
+			(at 27.94 35.052 90)
 			(effects
 				(font
@@
 	(symbol
 		(lib_id "power:+12V")
-		(at 22.86 36.83 0)
+		(at 23.495 29.21 0)
 		(unit 1)
 		(exclude_from_sim no)
@@
 		(dnp no)
 		(property "Reference" "#PWR012"
-			(at 22.86 40.64 0)
+			(at 23.495 33.02 0)
 			(effects
 				(font
@@
 		)
 		(property "Value" "+GLV"
-			(at 20.32 33.02 0)
+			(at 22.606 25.4 0)
 			(effects
 				(font
@@
 		)
 		(property "Footprint" ""
-			(at 22.86 36.83 0)
+			(at 23.495 29.21 0)
 			(effects
 				(font
@@
 		)
 		(property "Datasheet" ""
-			(at 22.86 36.83 0)
+			(at 23.495 29.21 0)
 			(effects
 				(font
@@
 		)
 		(property "Description" ""
-			(at 22.86 36.83 0)
+			(at 23.495 29.21 0)
 			(effects
 				(font
@@
 	)
 	(symbol
+		(lib_id "power:PWR_FLAG")
+		(at 23.495 30.48 270)
+		(unit 1)
+		(exclude_from_sim no)
+		(in_bom yes)
+		(on_board yes)
+		(dnp no)
+		(property "Reference" "#FLG04"
+			(at 25.4 30.48 0)
+			(effects
+				(font
+					(size 1.27 1.27)
+				)
+				(hide yes)
+			)
+		)
+		(property "Value" "PWR_FLAG"
+			(at 29.972 28.702 90)
+			(effects
+				(font
+					(size 1.27 1.27)
+				)
+			)
+		)
+		(property "Footprint" ""
+			(at 23.495 30.48 0)
+			(effects
+				(font
+					(size 1.27 1.27)
+				)
+				(hide yes)
+			)
+		)
+		(property "Datasheet" "~"
+			(at 23.495 30.48 0)
+			(effects
+				(font
+					(size 1.27 1.27)
+				)
+				(hide yes)
+			)
+		)
+		(property "Description" ""
+			(at 23.495 30.48 0)
+			(effects
+				(font
+					(size 1.27 1.27)
+				)
+			)
+		)
+		(pin "1"
+		)
+		(instances
+			(project "gps-mainboard"
+				(path "/de1c89a8-60ad-4219-8e58-e4b5538835d9"
+					(reference "#FLG04")
+					(unit 1)
+				)
+			)
+		)
+	)
+	(symbol
 		(lib_id "Device:NetTie_2")
 		(at 46.99 177.8 90)
@@
 					(unit 1)
 				)
-			)
-		)
-	)
-	(symbol
-		(lib_id "power:PWR_FLAG")
-		(at 73.66 126.365 0)
-		(unit 1)
-		(exclude_from_sim no)
-		(in_bom yes)
-		(on_board yes)
-		(dnp no)
-		(property "Reference" "#FLG04"
-			(at 73.66 124.46 0)
-			(effects
-				(font
-					(size 1.27 1.27)
-				)
-				(hide yes)
-			)
-		)
-		(property "Value" "PWR_FLAG"
-			(at 73.66 121.92 0)
-			(effects
-				(font
-					(size 1.27 1.27)
-				)
-			)
-		)
-		(property "Footprint" ""
-			(at 73.66 126.365 0)
-			(effects
-				(font
-					(size 1.27 1.27)
-				)
-				(hide yes)
-			)
-		)
-		(property "Datasheet" "~"
-			(at 73.66 126.365 0)
-			(effects
-				(font
-					(size 1.27 1.27)
-				)
-				(hide yes)
-			)
-		)
-		(property "Description" ""
-			(at 73.66 126.365 0)
-			(effects
-				(font
-					(size 1.27 1.27)
-				)
-			)
-		)
-		(pin "1"
-		)
-		(instances
-			(project "micromod-gps"
-				(path "/de1c89a8-60ad-4219-8e58-e4b5538835d9"
-					(reference "#FLG04")
-					(unit 1)
-				)
