File: sensor-hub/8Ch-Sensor-Hub.kicad_sch (KiCad schematic)
At the start: 33 parts, among them J1 Conn_ARM_JTAG_SWD_10, J2 Conn_01x04_Pin, J3 Conn_01x02, J4 Bottom_Left, J5 Top_Left, SW1 RESET, U2 STM32F105RBTx, Y1 ECS-250-10-47Q-CES-TR

Commit message: Tweak layout around connectors
Parts:
- J2: footprint SUFST:Molex_Micro-Fit_3.0_43045-0412_2x02_P3.00mm_Vertical -> Connector_Molex:Molex_Micro-Fit_3.0_43045-0400_2x02_P3.00mm_Horizontal
Changed lines of the file:
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@@
 			)
 		)
-		(property "Footprint" "SUFST:Molex_Micro-Fit_3.0_43045-0412_2x02_P3.00mm_Vertical"
+		(property "Footprint" "Connector_Molex:Molex_Micro-Fit_3.0_43045-0400_2x02_P3.00mm_Horizontal"
 			(at 50.8 200.66 0)
 			(effects
