File: rotary-switch/rotary-switch.kicad_sch (KiCad schematic)
At the start: 22 parts, among them J1 Conn_01x04_Socket, SW1 SW_Rotary_1x12, U1 TPS7B6925-Q1

Commit message: Update library from main
commit 70456059d4c90443398f32a8662464a85a6c0b63
Author: Ray Wang <114954263+saltyboi2995@users.noreply.github.com>
Date:   Tue Jul 7 09:34:59 2026 +0100

    July order BOM

commit 585a6f005b021ddb50761b87e6208ae7d3ed1ff8
Merge: 5be6b7a 38a5a96
Author: Ray Wang <114954263+saltyboi2995@users.noreply.github.com>
Date:   Mon Jun 15 15:35:29 2026 +0100

    Merge branch 'main' of https://github.com/sufst/pcb

commit 5be6b7ab45f952200be317d45337c550ed816c2e
Author: Ray Wang <114954263+saltyboi2995@users.noreply.github.com>
Date:   Mon Jun 15 15:35:03 2026 +0100

    Updated PCHG BOM for CCBOM

commit 38a5a96f5fb7a94bd63f2ebae4e014c2a68b46c7
Author: Ray Wang <114954263+saltyboi2995@users.noreply.github.com>
Date:   Mon Jun 15 15:33:49 2026 +0100

    Updated PCHG BOM for CCBOM

commit 5916207f99ec7c1dff868eef294f326f1008bcb4
Author: Agwld <eastman.adam1@gmail.com>
Date:   Sun Jun 14 15:30:49 2026 +0100

    correct TSMS naming on RSP pcb

commit aa40e7b71be525c58d68b60671a08eeeecb15947
Author: Ray Wang <114954263+saltyboi2995@users.noreply.github.com>
Date:   Sat Jun 13 13:35:19 2026 +0100

    Unarchive TEM

commit 4cfdd259bf584ef0bd9a0746033c9075a764595c
Author: Ray Wang <114954263+saltyboi2995@users.noreply.github.com>
Date:   Fri Jun 12 12:30:45 2026 +0100

    Sensor Hub 1.2.0 Release (#154)

    * progress from last week

    * temp update

    To find GND issue

    * Current Design 18/11/25

    Current agreed design at the time of EOS, by Adam and Ray contributions

    * Update library paths and clean up PCB net segments

    Replaced absolute library paths with project-relative variables in fp-lib-table and sym-lib-table for improved portability. Removed redundant or unnecessary traces.

    * Add fuses and update connector/capacitor references

    Added Device: Fuse symbols and instances to the schematic for overcurrent protection. Updated connector and capacitor reference designators and locations, and extended several nets to new co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
Parts:
- U1: value TPS7B6925-Q1 -> TPS7B6933-Q1; MPN TPS7B6925-Q1 -> TPS7B6933-Q1
Changed lines of the file:
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@@
 			)
 		)
-		(property "Value" "TPS7B6925-Q1"
+		(property "Value" "TPS7B6933-Q1"
 			(at 54.61 27.94 0)
 			(effects
@@
 			)
 		)
-		(property "MPN" "TPS7B6925-Q1"
+		(property "MPN" "TPS7B6933-Q1"
 			(at 54.61 33.02 0)
 			(effects
